File: Hardware/Digital board/Digital_board.sch (KiCad schematic (older format))
At the start: 255 parts, among them P1 1.8MHz osc, P2 SW_DIP9, P3 CONN_01X04, U1 7402, U10 74LS688, U100 74LS373, U101 74LS688, U102 74LS688, U103 74LS688, U104 74LS688, U105 4040, U106 4040, U107 4040, U108 4040, U109 74HCT02, U11 74LS688, U110 74LS688, U111 74LS688, U112 4040, U113 4040, U114 74LS688, U115 74LS688, U116 4040, U117 4040, U118 74LS373, U119 74LS373, U12 4040, U120 74LS373, U121 74LS373, U122 74LS32, U123 4040, U124 4040, U125 74LS541, U126 74LS541, U127 SST39SF020, U128 SST39SF020, U129 74LS30, U13 4040, U130 74LS30, U131 4040, U132 SST39SF020, U133 4040, U134 4040, U14 4040, U15 4040, U16 74LS541, U17 74LS541, U18 SST39SF020, U19 SST39SF020, U2 74LS373, U20 74LS30, U21 74LS30, U22 74HCT02, U23 74LS688, U24 74LS688, U25 4040, U26 4040, U27 74LS688, U28 74LS688, U29 4040, U3 74LS373, U30 4040, U31 4040, U32 74LS373, U33 74LS373, U34 74LS373, U35 74LS373, U36 74LS238, U37 74LS238, U38 74HC74, U39 74HC74, U4 74LS541, U40 74LS373, U41 74LS373, U42 74LS373, U43 74LS373, U44 74HC74, U46 74HC74, U47 74LS688, U48 74LS688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

Commit message: Connectors
Connectors for transfering signal to the analog board
Parts:
- removed U62, U64, U70, U71: 74HC74, symbol 74HC74
- added P?: CONN_02X32, symbol CONN_02X32
- added P?: CONN_02X20, symbol CONN_02X20
- added U? (x24): 74HC74, symbol 74HC74
Connections:
- net AD_db0: now also P?.33 (P33)
- net AD_db1: now also P?.35 (P35)
- net AD_db2: now also P?.37 (P37)
- net AD_db3: now also P?.39 (P39)
- net AD_db4: now also P?.2 (P2)
- net AD_db5: now also P?.4 (P4)
- net AD_db6: now also P?.6 (P6)
- net AD_db7: now also P?.8 (P8)
- net Amout0: now also P?.1 (P1)
- net Amout1: now also P?.3 (P3)
- net Amout10: now also P?.21 (P21), U?.5 (Q)
- net Amout11: now also P?.23 (P23), U?.9 (Q)
- net Amout12: now also P?.25 (P25), U?.5 (Q)
- net Amout13: now also P?.27 (P27), U?.9 (Q)
- net Amout14: now also P?.29 (P29), U?.5 (Q)
- net Amout15: now also P?.31 (P31), U?.9 (Q)
- net Amout2: now also P?.5 (P5)
- net Amout3: now also P?.7 (P7)
- net Amout4: now also P?.9 (P9)
- net Amout5: now also P?.11 (P11)
- net Amout6: now also P?.13 (P13)
- net Amout7: now also P?.15 (P15)
- net Amout8: now also P?.17 (P17), U?.5 (Q)
- net Amout9: now also P?.19 (P19), U?.9 (Q)
- net Av_amp0_C0: now also P?.1 (P1)
- net Av_amp0_C1: now also P?.9 (P9)
- net Av_amp0_C10: now also P?.18 (P18)
- net Av_amp0_C11: now also P?.26 (P26)
- net Av_amp0_C12: now also P?.34 (P34)
- net Av_amp0_C13: now also P?.42 (P42)
- net Av_amp0_C14: now also P?.50 (P50)
- net Av_amp0_C15: now also P?.58 (P58)
- net Av_amp0_C2: now also P?.17 (P17)
- net Av_amp0_C3: now also P?.25 (P25)
- net Av_amp0_C4: now also P?.33 (P33)
- net Av_amp0_C5: now also P?.41 (P41)
- net Av_amp0_C6: now also P?.49 (P49)
- net Av_amp0_C7: now also P?.57 (P57)
- net Av_amp0_C8: now also P?.2 (P2)
- net Av_amp0_C9: now also P?.10 (P10)
- net Av_amp1_C0: now also P?.3 (P3)
- net Av_amp1_C1: now also P?.11 (P11)
- net Av_amp1_C10: now also P?.20 (P20)
- net Av_amp1_C11: now also P?.28 (P28)
- net Av_amp1_C12: now also P?.36 (P36)
- net Av_amp1_C13: now also P?.44 (P44)
- net Av_amp1_C14: now also P?.52 (P52)
- net Av_amp1_C15: now also P?.60 (P60)
- net Av_amp1_C2: now also P?.19 (P19)
- net Av_amp1_C3: now also P?.27 (P27)
- net Av_amp1_C4: now also P?.35 (P35)
- net Av_amp1_C5: now also P?.43 (P43)
- net Av_amp1_C6: now also P?.51 (P51)
- net Av_amp1_C7: now also P?.59 (P59)
- net Av_amp1_C8: now also P?.4 (P4)
- net Av_amp1_C9: now also P?.12 (P12)
- net Av_amp2_C0: now also P?.5 (P5)
- net Av_amp2_C1: now also P?.13 (P13)
- net Av_amp2_C10: now also P?.22 (P22)
- net Av_amp2_C11: now also P?.30 (P30)
- net Av_amp2_C12: now also P?.38 (P38)
- net Av_amp2_C13: now also P?.46 (P46)
- net Av_amp2_C14: now also P?.54 (P54)
- net Av_amp2_C15: now also P?.62 (P62)
- net Av_amp2_C2: now also P?.21 (P21)
- net Av_amp2_C3: now also P?.29 (P29)
- net Av_amp2_C4: now also P?.37 (P37)
- net Av_amp2_C5: now also P?.45 (P45)
- net Av_amp2_C6: now also P?.53 (P53)
- net Av_amp2_C7: now also P?.61 (P61)
- net Av_amp2_C8: now also P?.6 (P6)
- net Av_amp2_C9: now also P?.14 (P14)
- net Av_amp3_C0: now also P?.7 (P7)
- net Av_amp3_C1: now also P?.15 (P15)
- net Av_amp3_C10: now also P?.24 (P24)
- net Av_amp3_C11: now also P?.32 (P32)
- net Av_amp3_C12: now also P?.40 (P40)
- net Av_amp3_C13: now also P?.48 (P48)
- net Av_amp3_C14: now also P?.56 (P56)
- net Av_amp3_C15: now also P?.64 (P64)
- net Av_amp3_C2: now also P?.23 (P23)
- net Av_amp3_C3: now also P?.31 (P31)
- net Av_amp3_C4: now also P?.39 (P39)
- net Av_amp3_C5: now also P?.47 (P47)
- net Av_amp3_C6: now also P?.55 (P55)
- net Av_amp3_C7: now also P?.63 (P63)
- net Av_amp3_C8: now also P?.8 (P8)
- net Av_amp3_C9: now also P?.16 (P16)
- net GND: now also U?.7 (GND), U?.7 (GND), U?.7 (GND), U?.7 (GND), U?.7 (GND), U?.7 (GND), U?.7 (GND), U?.7 (GND), U?.7 (GND), U?.7 (GND), U?.7 (GND), U?.7 (GND), U?.7 (GND), U?.7 (GND), U?.7 (GND), U?.7 (GND), U?.7 (GND), U?.7 (GND), U?.7 (GND), U?.7 (GND), U?.7 (GND), U?.7 (GND), U?.7 (GND), U?.7 (GND)
- net Rst_clk_audm10: now also U?.3 (Cp)
- net Rst_clk_audm11: now also U?.11 (Cp)
- net Rst_clk_audm12: now also U?.3 (Cp)
- net Rst_clk_audm13: now also U?.11 (Cp)
- net Rst_clk_audm14: now also U?.3 (Cp)
- net Rst_clk_audm15: now also U?.11 (Cp)
- net Rst_clk_audm8: now also U?.3 (Cp)
- net Rst_clk_audm9: now also U?.11 (Cp)
- net Rst_clk_audv0: now also U?.3 (Cp)
- net Rst_clk_audv1: now also U?.3 (Cp)
- net Rst_clk_audv10: now also U?.3 (Cp)
- net Rst_clk_audv11: now also U?.3 (Cp)
- net Rst_clk_audv12: now also U?.3 (Cp)
- net Rst_clk_audv13: now also U?.3 (Cp)
- net Rst_clk_audv14: now also U?.3 (Cp)
- net Rst_clk_audv15: now also U?.3 (Cp)
- net Rst_clk_audv2: now also U?.3 (Cp)
- net Rst_clk_audv3: now also U?.3 (Cp)
- net Rst_clk_audv4: now also U?.3 (Cp)
- net Rst_clk_audv5: now also U?.3 (Cp)
- net Rst_clk_audv6: now also U?.3 (Cp)
- net Rst_clk_audv7: now also U?.3 (Cp)
- net Rst_clk_audv8: now also U?.3 (Cp)
- net Rst_clk_audv9: now also U?.3 (Cp)
- net VCC: now also U?.1 (Cd), U?.1 (Cd), U?.1 (Cd), U?.1 (Cd), U?.1 (Cd), U?.1 (Cd), U?.1 (Cd), U?.1 (Cd), U?.1 (Cd), U?.1 (Cd), U?.1 (Cd), U?.1 (Cd), U?.1 (Cd), U?.1 (Cd), U?.1 (Cd), U?.1 (Cd), U?.1 (Cd), U?.1 (Cd), U?.1 (Cd), U?.1 (Cd), U?.10 (Sd), U?.10 (Sd), U?.10 (Sd), U?.10 (Sd), U?.13 (Cd), U?.13 (Cd), U?.13 (Cd), U?.13 (Cd), U?.14 (VCC), U?.14 (VCC), U?.14 (VCC), U?.14 (VCC), U?.14 (VCC), U?.14 (VCC), U?.14 (VCC), U?.14 (VCC), U?.14 (VCC), U?.14 (VCC), U?.14 (VCC), U?.14 (VCC), U?.14 (VCC), U?.14 (VCC), U?.14 (VCC), U?.14 (VCC), U?.14 (VCC), U?.14 (VCC), U?.14 (VCC), U?.14 (VCC), U?.14 (VCC), U?.14 (VCC), U?.14 (VCC), U?.14 (VCC), U?.4 (Sd), U?.4 (Sd), U?.4 (Sd), U?.4 (Sd), U?.4 (Sd), U?.4 (Sd), U?.4 (Sd), U?.4 (Sd), U?.4 (Sd), U?.4 (Sd), U?.4 (Sd), U?.4 (Sd), U?.4 (Sd), U?.4 (Sd), U?.4 (Sd), U?.4 (Sd), U?.4 (Sd), U?.4 (Sd), U?.4 (Sd), U?.4 (Sd)
- new net: U?.2 (D), U?.6 (~Q) (x20)
- new net: U?.12 (D), U?.8 (~Q) (x4)
- new net Avout0: P?.10 (P10), U?.5 (Q)
- new net Avout1: P?.12 (P12), U?.5 (Q)
- new net Avout10: P?.30 (P30), U?.5 (Q)
- new net Avout11: P?.32 (P32), U?.5 (Q)
- new net Avout12: P?.34 (P34), U?.5 (Q)
- new net Avout13: P?.36 (P36), U?.5 (Q)
- new net Avout14: P?.38 (P38), U?.5 (Q)
- new net Avout15: P?.40 (P40), U?.5 (Q)
- new net Avout2: P?.14 (P14), U?.5 (Q)
- new net Avout3: P?.16 (P16), U?.5 (Q)
- new net Avout4: P?.18 (P18), U?.5 (Q)
- new net Avout5: P?.20 (P20), U?.5 (Q)
- new net Avout6: P?.22 (P22), U?.5 (Q)
- new net Avout7: P?.24 (P24), U?.5 (Q)
- new net Avout8: P?.26 (P26), U?.5 (Q)
- new net Avout9: P?.28 (P28), U?.5 (Q)
Other:
- moved on the sheet: U38A, U38B, U39A, U39B, U44A, U44B, U46A, U46B

Commit message: ERC
Corrections after ERC pass
Parts:
- added P6: CONN_01X03, symbol CONN_01X03
- added P7: CONN_02X05, symbol CONN_02X05
- gave numbers to parts that had none: 117
Connections:
- net VDD is gone; now on net VCC: U105.16 (VDD), U106.16 (VDD), U107.16 (VDD), U108.16 (VDD), U112.16 (VDD), U113.16 (VDD), U116.16 (VDD), U117.16 (VDD), U12.16 (VDD), U123.16 (VDD), U124.16 (VDD), U13.16 (VDD), U131.16 (VDD), U133.16 (VDD), U134.16 (VDD), U137.16 (VDD), U139.16 (VDD), U14.16 (VDD), U149.16 (VDD), U15.16 (VDD), U151.16 (VDD), U153.16 (VDD), U156.16 (VDD), U157.16 (VDD), U160.16 (VDD), U169.16 (VDD), U172.16 (VDD), U174.16 (VDD), U177.16 (VDD), U182.16 (VDD), U183.16 (VDD), U184.16 (VDD), U186.16 (VDD), U192.16 (VDD), U198.16 (VDD), U212.16 (VDD), U213.16 (VDD), U216.16 (VDD), U220.16 (VDD), U222.16 (VDD), U226.16 (VDD), U227.16 (VDD), U228.16 (VDD), U232.16 (VDD), U238.16 (VDD), U240.16 (VDD), U241.16 (VDD), U25.16 (VDD), U26.16 (VDD), U29.16 (VDD), U30.16 (VDD), U31.16 (VDD), U51.16 (VDD), U52.16 (VDD), U53.16 (VDD), U54.16 (VDD), U58.16 (VDD), U59.16 (VDD), U63.16 (VDD), U64.16 (VDD), U65.16 (VDD), U7.16 (VDD), U71.16 (VDD), U80.16 (VDD), U81.16 (VDD), U82.16 (VDD), U83.16 (VDD), U87.16 (VDD), U88.16 (VDD), U91.16 (VDD), U92.16 (VDD)
- net AV_db10: now also U125.16 (Y2)
- net AV_db11: now also U125.15 (Y3)
- net AV_db12: now also U125.14 (Y4)
- net AV_db13: now also U125.13 (Y5)
- net AV_db14: now also U125.12 (Y6)
- net AV_db15: now also U125.11 (Y7)
- net AV_db8: now also U125.18 (Y0)
- net AV_db9: now also U125.17 (Y1)
- net Amout11: now also U197.5 (Q); no longer U197.9 (Q)
- net Amout13: now also U208.5 (Q); no longer U208.9 (Q)
- net Amout9: now also U179.5 (Q); no longer U179.9 (Q)
- net Avout0: now also U170.9 (Q); no longer U170.5 (Q)
- net Avout1: now also U181.9 (Q); no longer U181.5 (Q)
- net Avout10: now also U208.9 (Q); no longer U208.5 (Q)
- net Avout2: now also U191.9 (Q); no longer U191.5 (Q)
- net Avout3: now also U199.9 (Q); no longer U199.5 (Q)
- net Avout4: now also U204.9 (Q); no longer U204.5 (Q)
- net Avout5: now also U210.9 (Q); no longer U210.5 (Q)
- net Avout6: now also U179.9 (Q); no longer U179.5 (Q)
- net Avout7: now also U189.9 (Q); no longer U189.5 (Q)
- net Avout8: now also U197.9 (Q); no longer U197.5 (Q)
- net Avout9: now also U202.9 (Q); no longer U202.5 (Q)
- net Clk_main6: now also P6.2 (P2)
- net Clk_main7: now also P6.1 (P1)
- net GND: now also P6.3 (P3)
- net Master_reset: now also P7.1 (P1)
- net Rst_clk_audm11: now also U197.3 (Cp); no longer U197.11 (Cp)
- net Rst_clk_audm13: now also U208.3 (Cp); no longer U208.11 (Cp)
- net Rst_clk_audm9: now also U179.3 (Cp); no longer U179.11 (Cp)
- net Rst_clk_audv0: now also U170.11 (Cp); no longer U170.3 (Cp)
- net Rst_clk_audv1: now also U136.4, U181.11 (Cp); no longer U136.1, U181.3 (Cp)
- net Rst_clk_audv10: now also U208.11 (Cp), U219.4; no longer U208.3 (Cp), U219.1
- net Rst_clk_audv11: now also U219.13; no longer U219.1
- net Rst_clk_audv12: now also U219.10; no longer U219.1
- net Rst_clk_audv13: now also U180.10; no longer U180.1
- net Rst_clk_audv15: now also U180.13; no longer U180.1
- net Rst_clk_audv2: now also U136.10, U191.11 (Cp); no longer U136.1, U191.3 (Cp)
- net Rst_clk_audv3: now also U136.13, U199.11 (Cp); no longer U136.1, U199.3 (Cp)
- net Rst_clk_audv4: now also U204.11 (Cp); no longer U204.3 (Cp)
- net Rst_clk_audv5: now also U155.4, U210.11 (Cp); no longer U155.1, U210.3 (Cp)
- net Rst_clk_audv6: now also U155.10, U179.11 (Cp); no longer U155.1, U179.3 (Cp)
- net Rst_clk_audv7: now also U155.13, U189.11 (Cp); no longer U155.1, U189.3 (Cp)
- net Rst_clk_audv8: now also U180.4, U197.11 (Cp); no longer U180.1, U197.3 (Cp)
- net Rst_clk_audv9: now also U202.11 (Cp); no longer U202.3 (Cp)
- net VCC: now also U170.10 (Sd), U170.13 (Cd), U179.1 (Cd), U179.10 (Sd), U179.13 (Cd), U179.4 (Sd), U181.10 (Sd), U181.13 (Cd), U189.10 (Sd), U189.13 (Cd), U191.10 (Sd), U191.13 (Cd), U197.1 (Cd), U197.10 (Sd), U197.13 (Cd), U197.4 (Sd), U199.10 (Sd), U199.13 (Cd), U202.10 (Sd), U202.13 (Cd), U204.10 (Sd), U204.13 (Cd), U208.1 (Cd), U208.10 (Sd), U208.13 (Cd), U208.4 (Sd), U210.10 (Sd), U210.13 (Cd); no longer U170.1 (Cd), U170.4 (Sd), U179.1 (Cd), U179.10 (Sd), U179.13 (Cd), U179.4 (Sd), U181.1 (Cd), U181.4 (Sd), U189.1 (Cd), U189.4 (Sd), U191.1 (Cd), U191.4 (Sd), U197.1 (Cd), U197.10 (Sd), U197.13 (Cd), U197.4 (Sd), U199.1 (Cd), U199.4 (Sd), U202.1 (Cd), U202.4 (Sd), U204.1 (Cd), U204.4 (Sd), U208.1 (Cd), U208.10 (Sd), U208.13 (Cd), U208.4 (Sd), U210.1 (Cd), U210.4 (Sd)
- net Voice_reset_blank: now also P7.2 (P2)
- net Voice_select0: now also P7.3 (P3)
- net Voice_select1: now also P7.5 (P5)
- net Voice_select2: now also P7.7 (P7)
- net at U141.19 (P=R): now also U136.5; no longer U136.2
- net at U135.19 (P=R): now also U136.6; no longer U136.3
- net at U158.19 (P=R): now also U136.8; no longer U136.2
- net at U150.19 (P=R): now also U136.9; no longer U136.3
- net at U159.19 (P=R): now also U136.11; no longer U136.2
- net at U152.19 (P=R): now also U136.12; no longer U136.3
- net at U185.19 (P=R): now also U155.5; no longer U155.2
- net at U171.19 (P=R): now also U155.6; no longer U155.3
- net at U188.19 (P=R): now also U155.8; no longer U155.2
- net at U173.19 (P=R): now also U155.9; no longer U155.3
- net at U229.19 (P=R): now also U180.8; no longer U180.2
- net at U214.19 (P=R): now also U180.9; no longer U180.3
- net at U190.19 (P=R): now also U155.11; no longer U155.2
- net at U175.19 (P=R): now also U155.12; no longer U155.3
- net at U230.19 (P=R): now also U180.11; no longer U180.2
- net at U215.19 (P=R): now also U180.12; no longer U180.3
- net at U201.19 (P=R): now also U180.5; no longer U180.2
- net at U187.19 (P=R): now also U180.6; no longer U180.3
- net at U242.19 (P=R): now also U219.11; no longer U219.2
- net at U225.19 (P=R): now also U219.12; no longer U219.3
- net at U236.19 (P=R): now also U219.8; no longer U219.2
- net at U221.19 (P=R): now also U219.9; no longer U219.3
- net at U223.19 (P=R): now also U219.5; no longer U219.2
- net at U224.19 (P=R): now also U219.6; no longer U219.3
- new net: U208.2 (D), U208.6 (~Q)
- new net: U179.2 (D), U179.6 (~Q)
- new net: U197.2 (D), U197.6 (~Q)
- new net: U170.12 (D), U170.8 (~Q)
- new net: U181.12 (D), U181.8 (~Q)
- new net: U191.12 (D), U191.8 (~Q)
- new net: U199.12 (D), U199.8 (~Q)
- new net: U179.12 (D), U179.8 (~Q)
- new net: U189.12 (D), U189.8 (~Q)
- new net: U197.12 (D), U197.8 (~Q)
- new net: U202.12 (D), U202.8 (~Q)
- new net: U204.12 (D), U204.8 (~Q)
- new net: U210.12 (D), U210.8 (~Q)
- new net: U208.12 (D), U208.8 (~Q)
- no-connect marks 660 -> 670
Other:
- moved on the sheet: P2, R1, R2, R24, R25

Commit message: Components association
Parts:
- P1: footprint (none) -> Sockets_DIP:DIP-14__300
- P2: footprint (none) -> Sockets_DIP:DIP-18__300
- P3: footprint (none) -> Socket_Strips:Socket_Strip_Straight_1x04
- P4: footprint (none) -> Socket_Strips:Socket_Strip_Straight_2x32
- P5: footprint (none) -> Socket_Strips:Socket_Strip_Straight_2x20
- P6: footprint (none) -> Socket_Strips:Socket_Strip_Straight_1x03
- P7: footprint (none) -> Socket_Strips:Socket_Strip_Straight_2x05
- R1, R2, R24, R25: footprint (none) -> Resistors_SMD:R_0805_HandSoldering
- U1: footprint (none) -> Sockets_DIP:DIP-8__300
- U10, U11, U16, U17, U2, U3, U4, U5, U6, U8, U9: footprint (none) -> Sockets_DIP:DIP-20__300
- U12, U13, U14, U15, U7: footprint (none) -> Sockets_DIP:DIP-16__300
- U18, U19: footprint (none) -> Sockets_DIP:DIP-32__600

Commit message: Decoupling cap
Parts:
- added C? (x40): 1µ, symbol C_Small
- added C? (x2): 47µ, symbol CP_Small
- added C? (x260): 22n, symbol C_Small
- added unit 3 of U138
- added unit 4 of U138
- added unit 2 of U138
- U100, U101, U102, U103, U104, U110, U111, U114, U115, U118, U119, U120, U121, U125, U126, U135, U140, U141, U143, U144, U146, U147, U148, U150, U152, U154, U158, U159, U161, U162, U163, U164, U165, U166, U167, U168, U171, U173, U175, U176, U178, U185, U187, U188, U190, U193, U194, U195, U196, U200, U201, U203, U205, U206, U207, U209, U211, U214, U215, U217, U221, U223, U224, U225, U229, U23, U230, U231, U233, U234, U235, U236, U237, U239, U24, U242, U243, U244, U27, U28, U32, U33, U34, U35, U40, U41, U42, U43, U45, U47, U48, U49, U50, U56, U57, U60, U61, U62, U66, U67, U68, U69, U70, U72, U73, U74, U75, U76, U77, U78, U79, U85, U86, U89, U90, U93, U94, U95, U96, U97, U98, U99: footprint (none) -> Sockets_DIP:DIP-20__300
- U105, U106, U107, U108, U112, U113, U116, U117, U123, U124, U131, U133, U134, U137, U139, U142, U145, U149, U151, U153, U156, U157, U160, U169, U172, U174, U177, U182, U183, U184, U186, U192, U198, U212, U213, U216, U220, U222, U226, U227, U228, U232, U238, U240, U241, U25, U26, U29, U30, U31, U36, U37, U51, U52, U53, U54, U58, U59, U63, U64, U65, U71, U80, U81, U82, U83, U87, U88, U91, U92: footprint (none) -> Sockets_DIP:DIP-16__300
- U109, U129, U130, U136, U138, U155, U170, U179, U180, U181, U189, U191, U197, U199, U20, U202, U204, U208, U21, U210, U218, U219, U22, U38, U39, U44, U46, U55, U84: footprint (none) -> Sockets_DIP:DIP-14__300
- U122: footprint (none) -> Sockets_DIP:DIP-8__300
- U127, U128, U132: footprint (none) -> Sockets_DIP:DIP-32__600
Connections:
- net GND: now also C?.2, C?.2, C?.2, C?.2, C?.2, C?.2, C?.2, C?.2, C?.2, C?.2, C?.2, C?.2, C?.2, C?.2, C?.2, C?.2, C?.2, C?.2, C?.2, C?.2, C?.2, C?.2, C?.2, C?.2, C?.2, C?.2, C?.2, C?.2, C?.2, C?.2, C?.2, C?.2, C?.2, C?.2, C?.2, C?.2, C?.2, C?.2, C?.2, C?.2, C?.2, C?.2, C?.2, C?.2, C?.2, C?.2, C?.2, C?.2, C?.2, C?.2, C?.2, C?.2, C?.2, C?.2, C?.2, C?.2, C?.2, C?.2, C?.2, C?.2, C?.2, C?.2, C?.2, C?.2, C?.2, C?.2, C?.2, C?.2, C?.2, C?.2, C?.2, C?.2, C?.2, C?.2, C?.2, C?.2, C?.2, C?.2, C?.2, C?.2, C?.2, C?.2, C?.2, C?.2, C?.2, C?.2, C?.2, C?.2, C?.2, C?.2, C?.2, C?.2, C?.2, C?.2, C?.2, C?.2, C?.2, C?.2, C?.2, C?.2, C?.2, C?.2, C?.2, C?.2, C?.2, C?.2, C?.2, C?.2, C?.2, C?.2, C?.2, C?.2, C?.2, C?.2, C?.2, C?.2, C?.2, C?.2, C?.2, C?.2, C?.2, C?.2, C?.2, C?.2, C?.2, C?.2, C?.2, C?.2, C?.2, C?.2, C?.2, C?.2, C?.2, C?.2, C?.2, C?.2, C?.2, C?.2, C?.2, C?.2, C?.2, C?.2, C?.2, C?.2, C?.2, C?.2, C?.2, C?.2, C?.2, C?.2, C?.2, C?.2, C?.2, C?.2, C?.2, C?.2, C?.2, C?.2, C?.2, C?.2, C?.2, C?.2, C?.2, C?.2, C?.2, C?.2, C?.2, C?.2, C?.2, C?.2, C?.2, C?.2, C?.2, C?.2, C?.2, C?.2, C?.2, C?.2, C?.2, C?.2, C?.2, C?.2, C?.2, C?.2, C?.2, C?.2, C?.2, C?.2, C?.2, C?.2, C?.2, C?.2, C?.2, C?.2, C?.2, C?.2, C?.2, C?.2, C?.2, C?.2, C?.2, C?.2, C?.2, C?.2, C?.2, C?.2, C?.2, C?.2, C?.2, C?.2, C?.2, C?.2, C?.2, C?.2, C?.2, C?.2, C?.2, C?.2, C?.2, C?.2, C?.2, C?.2, C?.2, C?.2, C?.2, C?.2, C?.2, C?.2, C?.2, C?.2, C?.2, C?.2, C?.2, C?.2, C?.2, C?.2, C?.2, C?.2, C?.2, C?.2, C?.2, C?.2, C?.2, C?.2, C?.2, C?.2, C?.2, C?.2, C?.2, C?.2, C?.2, C?.2, C?.2, C?.2, C?.2, C?.2, C?.2, C?.2, C?.2, C?.2, C?.2, C?.2, C?.2, C?.2, C?.2, C?.2, C?.2, C?.2, C?.2, C?.2, C?.2, C?.2, C?.2, C?.2, C?.2, C?.2, C?.2, C?.2, C?.2, C?.2, C?.2, C?.2, C?.2, C?.2, C?.2, C?.2, C?.2, C?.2, C?.2, C?.2, C?.2, C?.2, C?.2, C?.2, C?.2, C?.2, C?.2, C?.2, C?.2, C?.2, C?.2, C?.2, U138.10, U138.12, U138.13, U138.4, U138.5, U138.7 (GND), U138.7 (GND), U138.7 (GND), U138.9; no longer U131.11 (Reset), U31.11 (Reset)
- net Master_reset: now also U131.11 (Reset), U31.11 (Reset)
- net VCC: now also C?.1, C?.1, C?.1, C?.1, C?.1, C?.1, C?.1, C?.1, C?.1, C?.1, C?.1, C?.1, C?.1, C?.1, C?.1, C?.1, C?.1, C?.1, C?.1, C?.1, C?.1, C?.1, C?.1, C?.1, C?.1, C?.1, C?.1, C?.1, C?.1, C?.1, C?.1, C?.1, C?.1, C?.1, C?.1, C?.1, C?.1, C?.1, C?.1, C?.1, C?.1, C?.1, C?.1, C?.1, C?.1, C?.1, C?.1, C?.1, C?.1, C?.1, C?.1, C?.1, C?.1, C?.1, C?.1, C?.1, C?.1, C?.1, C?.1, C?.1, C?.1, C?.1, C?.1, C?.1, C?.1, C?.1, C?.1, C?.1, C?.1, C?.1, C?.1, C?.1, C?.1, C?.1, C?.1, C?.1, C?.1, C?.1, C?.1, C?.1, C?.1, C?.1, C?.1, C?.1, C?.1, C?.1, C?.1, C?.1, C?.1, C?.1, C?.1, C?.1, C?.1, C?.1, C?.1, C?.1, C?.1, C?.1, C?.1, C?.1, C?.1, C?.1, C?.1, C?.1, C?.1, C?.1, C?.1, C?.1, C?.1, C?.1, C?.1, C?.1, C?.1, C?.1, C?.1, C?.1, C?.1, C?.1, C?.1, C?.1, C?.1, C?.1, C?.1, C?.1, C?.1, C?.1, C?.1, C?.1, C?.1, C?.1, C?.1, C?.1, C?.1, C?.1, C?.1, C?.1, C?.1, C?.1, C?.1, C?.1, C?.1, C?.1, C?.1, C?.1, C?.1, C?.1, C?.1, C?.1, C?.1, C?.1, C?.1, C?.1, C?.1, C?.1, C?.1, C?.1, C?.1, C?.1, C?.1, C?.1, C?.1, C?.1, C?.1, C?.1, C?.1, C?.1, C?.1, C?.1, C?.1, C?.1, C?.1, C?.1, C?.1, C?.1, C?.1, C?.1, C?.1, C?.1, C?.1, C?.1, C?.1, C?.1, C?.1, C?.1, C?.1, C?.1, C?.1, C?.1, C?.1, C?.1, C?.1, C?.1, C?.1, C?.1, C?.1, C?.1, C?.1, C?.1, C?.1, C?.1, C?.1, C?.1, C?.1, C?.1, C?.1, C?.1, C?.1, C?.1, C?.1, C?.1, C?.1, C?.1, C?.1, C?.1, C?.1, C?.1, C?.1, C?.1, C?.1, C?.1, C?.1, C?.1, C?.1, C?.1, C?.1, C?.1, C?.1, C?.1, C?.1, C?.1, C?.1, C?.1, C?.1, C?.1, C?.1, C?.1, C?.1, C?.1, C?.1, C?.1, C?.1, C?.1, C?.1, C?.1, C?.1, C?.1, C?.1, C?.1, C?.1, C?.1, C?.1, C?.1, C?.1, C?.1, C?.1, C?.1, C?.1, C?.1, C?.1, C?.1, C?.1, C?.1, C?.1, C?.1, C?.1, C?.1, C?.1, C?.1, C?.1, C?.1, C?.1, C?.1, C?.1, C?.1, C?.1, C?.1, C?.1, C?.1, C?.1, C?.1, C?.1, C?.1, C?.1, C?.1, C?.1, C?.1, C?.1, C?.1, C?.1, C?.1, C?.1, C?.1, C?.1, C?.1, C?.1, C?.1, C?.1, C?.1, C?.1, C?.1, C?.1, C?.1, U138.14 (VCC), U138.14 (VCC), U138.14 (VCC)
- no-connect marks 670 -> 673

Commit message: PCB
Parts:
- removed U1: 7402, Sockets_DIP:DIP-8__300, symbol 7402
- added U1: 74HCT02, Sockets_DIP:DIP-14__300, symbol 74HCT02
- C1, C10, C100, C101, C102, C103, C104, C105, C106, C107, C108, C109, C11, C110, C111, C112, C113, C114, C115, C116, C117, C118, C119, C12, C120, C121, C122, C123, C124, C125, C126, C127, C128, C129, C13, C130, C131, C132, C133, C134, C135, C136, C137, C138, C139, C14, C140, C141, C142, C143, C144, C145, C146, C147, C148, C149, C15, C150, C151, C152, C153, C154, C155, C156, C157, C158, C159, C16, C160, C161, C162, C163, C164, C165, C166, C167, C168, C169, C17, C170, C171, C172, C173, C174, C175, C176, C177, C178, C179, C18, C180, C181, C182, C183, C184, C185, C186, C187, C188, C189, C19, C190, C191, C192, C193, C194, C195, C196, C197, C198, C199, C2, C20, C200, C21, C22, C23, C24, C243, C244, C245, C246, C247, C248, C249, C25, C250, C251, C252, C253, C254, C255, C256, C257, C258, C259, C26, C260, C261, C262, C263, C264, C265, C266, C267, C268, C269, C27, C270, C271, C272, C273, C274, C275, C276, C277, C278, C279, C28, C280, C281, C282, C283, C284, C285, C286, C287, C288, C289, C29, C290, C291, C292, C293, C294, C295, C296, C297, C298, C299, C3, C30, C300, C301, C302, C31, C32, C33, C34, C35, C36, C37, C38, C39, C4, C40, C41, C42, C43, C44, C45, C46, C47, C48, C49, C5, C50, C51, C52, C53, C54, C55, C56, C57, C58, C59, C6, C60, C61, C62, C63, C64, C65, C66, C67, C68, C69, C7, C70, C71, C72, C73, C74, C75, C76, C77, C78, C79, C8, C80, C81, C82, C83, C84, C85, C86, C87, C88, C89, C9, C90, C91, C92, C93, C94, C95, C96, C97, C98, C99: renamed from C?; footprint (none) -> Capacitors_SMD:C_0603_HandSoldering
- C201, C202: renamed from C?; footprint (none) -> Capacitors_SMD:C_1206_HandSoldering
- C203, C204, C205, C206, C207, C208, C209, C210, C211, C212, C213, C214, C215, C216, C217, C218, C219, C220, C221, C222, C223, C224, C225, C226, C227, C228, C229, C230, C231, C232, C233, C234, C235, C236, C237, C238, C239, C240, C241, C242: renamed from C?; footprint (none) -> Capacitors_SMD:C_0805_HandSoldering
- U122: footprint Sockets_DIP:DIP-8__300 -> Sockets_DIP:DIP-14__300
Connections:
- net GND: now also U1.11, U1.12, U1.7 (GND), U1.7 (GND), U1.7 (GND), U1.7 (GND), U1.8, U1.9
- net Rst_audV_1: now also U1.5
- net Rst_audV_2: now also U1.6
- net Rst_aud_1: now also U1.2
- net Rst_aud_2: now also U1.3
- net VCC: now also U1.14 (VCC), U1.14 (VCC), U1.14 (VCC), U1.14 (VCC)
- net at U122.1: now also U1.1
- net at U122.4: now also U1.4
- no-connect marks 673 -> 675

Commit message: Removed the fm synthesis
Removed the fm synthesis to keep project manageable on the remaining
time (<2month)
Parts:
- removed C1, C10, C100, C101, C102, C103, C104, C105, C106, C107, C108, C109, C11, C110, C111, C112, C113, C114, C115, C116, C117, C118, C119, C12, C120, C121, C122, C123, C124, C125, C126, C127, C128, C129, C13, C130, C131, C132, C133, C134, C135, C136, C137, C138, C139, C14, C140, C141, C142, C143, C144, C145, C146, C147, C148, C149, C15, C150, C151, C152, C153, C154, C155, C156, C157, C158, C159, C16, C160, C161, C162, C163, C164, C165, C166, C167, C168, C169, C17, C170, C171, C172, C173, C174, C175, C176, C177, C178, C179, C18, C180, C181, C182, C183, C184, C185, C186, C187, C188, C189, C19, C190, C191, C192, C193, C194, C195, C196, C197, C198, C199, C2, C20, C200, C21, C22, C23, C24, C243, C244, C245, C246, C247, C248, C249, C25, C250, C251, C252, C253, C254, C255, C256, C257, C258, C259, C26, C260, C261, C262, C263, C264, C265, C266, C267, C268, C269, C27, C270, C271, C272, C273, C274, C275, C276, C277, C278, C279, C28, C280, C281, C282, C283, C284, C285, C286, C287, C288, C289, C29, C290, C291, C292, C293, C294, C295, C296, C297, C298, C299, C3, C30, C300, C301, C302, C31, C32, C33, C34, C35, C36, C37, C38, C39, C4, C40, C41, C42, C43, C44, C45, C46, C47, C48, C49, C5, C50, C51, C52, C53, C54, C55, C56, C57, C58, C59, C6, C60, C61, C62, C63, C64, C65, C66, C67, C68, C69, C7, C70, C71, C72, C73, C74, C75, C76, C77, C78, C79, C8, C80, C81, C82, C83, C84, C85, C86, C87, C88, C89, C9, C90, C91, C92, C93, C94, C95, C96, C97, C98, C99: 22n, Capacitors_SMD:C_0603_HandSoldering, symbol C_Small
- removed P2: SW_DIP9, Sockets_DIP:DIP-18__300, symbol DIL18
- removed P4: CONN_02X32, Socket_Strips:Socket_Strip_Straight_2x32, symbol CONN_02X32
- removed P5: CONN_02X20, Socket_Strips:Socket_Strip_Straight_2x20, symbol CONN_02X20
- removed R1, R2, R24, R25: 100k, Resistors_SMD:R_0805_HandSoldering, symbol R
- removed U1, U109, U136, U155, U180, U219, U22, U55, U84: 74HCT02, Sockets_DIP:DIP-14__300, symbol 74HCT02
- removed U10, U101, U102, U103, U104, U11, U110, U111, U114, U115, U135, U140, U141, U150, U152, U154, U158, U159, U162, U171, U173, U175, U178, U185, U187, U188, U190, U196, U201, U214, U215, U217, U221, U223, U224, U225, U229, U23, U230, U231, U236, U24, U242, U27, U28, U47, U48, U49, U50, U56, U57, U60, U61, U70, U76, U77, U78, U79, U8, U85, U86, U89, U9, U90: 74LS688, Sockets_DIP:DIP-20__300, symbol 74LS688
- removed U100, U118, U119, U120, U121, U143, U144, U146, U147, U161, U163, U164, U165, U166, U167, U168, U176, U193, U194, U195, U2, U200, U203, U205, U206, U207, U209, U211, U233, U234, U235, U237, U239, U243, U244, U3, U32, U33, U34, U35, U40, U41, U42, U43, U45, U5, U6, U62, U66, U67, U68, U69, U72, U73, U74, U75, U93, U94, U95, U96, U97, U98, U99: 74LS373, Sockets_DIP:DIP-20__300, symbol 74LS373
- removed U105, U106, U107, U108, U112, U113, U116, U117, U12, U123, U13, U137, U139, U14, U149, U15, U151, U153, U156, U157, U160, U169, U172, U174, U177, U182, U183, U184, U186, U192, U198, U212, U213, U216, U220, U222, U226, U227, U228, U232, U238, U240, U241, U25, U26, U29, U30, U31, U51, U52, U53, U54, U58, U59, U63, U64, U65, U7, U71, U80, U81, U82, U83, U87, U88, U91, U92: 4040, Sockets_DIP:DIP-16__300, symbol 4040
- removed unit 1 of U122
- removed U125, U16, U17: 74LS541, Sockets_DIP:DIP-20__300, symbol 74LS541
- removed U127, U132, U18, U19: SST39SF020, Sockets_DIP:DIP-32__600, symbol SST39SF020
- removed U129, U130, U20, U21: 74LS30, Sockets_DIP:DIP-14__300, symbol 74LS30
- removed U142, U145, U36, U37: 74LS238, Sockets_DIP:DIP-16__300, symbol 74LS138
- removed U170, U179, U181, U189, U191, U197, U199, U202, U204, U208, U210, U218, U38, U39, U44, U46: 74HC74, Sockets_DIP:DIP-14__300, symbol 74HC74
- added U? (x4): 74LS21, symbol 74LS21
- added U?: DAC08, symbol DAC08
- added U?: Dip-mem_2Mx8b, symbol Dip-mem_2Mx8b
- added U?: 74LS373, Sockets_DIP:DIP-20__300, symbol 74LS373
- added U?: 74LS32, Sockets_DIP:DIP-14__300, symbol 74LS32
- P1: value 1.8MHz osc -> 32kHz osc
Connections:
- net labels added: Rst_audM, Rst_audV
- net labels removed: A0_aud_m, A1_aud_m, A2_aud_m, A3_aud_m, AD_db0, AD_db1, AD_db2, AD_db3, AD_db4, AD_db5, AD_db6, AD_db7, AM_db10, AM_db11, AM_db12, AM_db13, AM_db14, AM_db15, AM_db8, AM_db9, Amout0, Amout1, Amout10, Amout11, Amout12, Amout13, Amout14, Amout15, Amout2, Amout3, Amout4, Amout5, Amout6, Amout7, Amout8, Amout9, Av_amp0_C0, Av_amp0_C1, Av_amp0_C10, Av_amp0_C11, Av_amp0_C12, Av_amp0_C13, Av_amp0_C14, Av_amp0_C15, Av_amp0_C2, Av_amp0_C3, Av_amp0_C4, Av_amp0_C5, Av_amp0_C6, Av_amp0_C7, Av_amp0_C8, Av_amp0_C9, Av_amp1_C0, Av_amp1_C1, Av_amp1_C10, Av_amp1_C11, Av_amp1_C12, Av_amp1_C13, Av_amp1_C14, Av_amp1_C15, Av_amp1_C2, Av_amp1_C3, Av_amp1_C4, Av_amp1_C5, Av_amp1_C6, Av_amp1_C7, Av_amp1_C8, Av_amp1_C9, Av_amp2_C0, Av_amp2_C1, Av_amp2_C10, Av_amp2_C11, Av_amp2_C12, Av_amp2_C13, Av_amp2_C14, Av_amp2_C15, Av_amp2_C2, Av_amp2_C3, Av_amp2_C4, Av_amp2_C5, Av_amp2_C6, Av_amp2_C7, Av_amp2_C8, Av_amp2_C9, Av_amp3_C0, Av_amp3_C1, Av_amp3_C10, Av_amp3_C11, Av_amp3_C12, Av_amp3_C13, Av_amp3_C14, Av_amp3_C15, Av_amp3_C2, Av_amp3_C3, Av_amp3_C4, Av_amp3_C5, Av_amp3_C6, Av_amp3_C7, Av_amp3_C8, Av_amp3_C9, Avout0, Avout1, Avout10, Avout11, Avout12, Avout13, Avout14, Avout15, Avout2, Avout3, Avout4, Avout5, Avout6, Avout7, Avout8, Avout9, BS1, BS2, BS3, BS4, BS5, BS6, BS7, BS8, BS9, Chm_0, Chm_1, Chm_10, Chm_11, Chm_12, Chm_13, Chm_14, Chm_15, Chm_2, Chm_3, Chm_4, Chm_5, Chm_6, Chm_7, Chm_8, Chm_9, Chv_0, Chv_1, Chv_10, Chv_11, Chv_12, Chv_13, Chv_14, Chv_15, Chv_2, Chv_3, Chv_4, Chv_5, Chv_6, Chv_7, Chv_8, Chv_9, Clk_aud_data, M_reset, Rst_audV_1, Rst_audV_2, Rst_clk_audm0, Rst_clk_audm1, Rst_clk_audm10, Rst_clk_audm11, Rst_clk_audm12, Rst_clk_audm13, Rst_clk_audm14, Rst_clk_audm15, Rst_clk_audm2, Rst_clk_audm3, Rst_clk_audm4, Rst_clk_audm5, Rst_clk_audm6, Rst_clk_audm7, Rst_clk_audm8, Rst_clk_audm9, Rst_clk_audv0, Rst_clk_audv1, Rst_clk_audv10, Rst_clk_audv11, Rst_clk_audv12, Rst_clk_audv13, Rst_clk_audv14, Rst_clk_audv15, Rst_clk_audv2, Rst_clk_audv3, Rst_clk_audv4, Rst_clk_audv5, Rst_clk_audv6, Rst_clk_audv7, Rst_clk_audv8, Rst_clk_audv9
- wire segments 4394 -> 425
- no-connect marks 675 -> 46
Other:
- moved on the sheet: U122B, U124, U126, U128, U131, U133, U134, U138A, U138B, U138C, U138D, U148

Commit message: Update
Parts:
- removed P6: CONN_01X03, Socket_Strips:Socket_Strip_Straight_1x03, symbol CONN_01X03
- removed P7: CONN_02X05, Socket_Strips:Socket_Strip_Straight_2x05, symbol CONN_02X05
- added P?: DIL18, symbol DIL18
- added U?: 4040, Sockets_DIP:DIP-16__300, symbol 4040
- added U? (x2): 74HC74, symbol 74HC74
- added U?: 74LS688, symbol 74LS688
- added U?: 74LS32, Sockets_DIP:DIP-14__300, symbol 74LS32
Connections:
- net labels added: Clk_divb0, Clk_divb1, Clk_divb10, Clk_divb11, Clk_divb12, Clk_divb13, Clk_divb14, Clk_divb15, Clk_divb16, Clk_divb17, Clk_divb18, Clk_divb19, Clk_divb2, Clk_divb20, Clk_divb3, Clk_divb4, Clk_divb5, Clk_divb6, Clk_divb7, Clk_divb8, Clk_divb9, Rst_Gam
- net labels removed: AV_db10, AV_db11, AV_db12, AV_db13, AV_db14, AV_db15, AV_db8, AV_db9, Rst_aud_1, Rst_aud_2
- wire segments 425 -> 308
- no-connect marks 46 -> 41
Other:
- moved on the sheet: U133, U134, U138B, U148, U?, U?A, U?B

Commit message: Schematic ERC corrections
Parts:
- removed C219, C220, C221, C222, C224, C225, C226, C227, C228, C229, C230, C231, C232, C233, C234, C235, C236, C237, C238, C239, C240, C241, C242: 1µ, Capacitors_SMD:C_0805_HandSoldering, symbol C_Small
- removed U126: 74LS541, Sockets_DIP:DIP-20__300, symbol 74LS541
- removed U?: DAC08, symbol DAC08
- removed U?: 4040, Sockets_DIP:DIP-16__300, symbol 4040
- removed U? (x2): 74HC74, symbol 74HC74
- removed U?: 74LS688, symbol 74LS688
- added C11, C12, C14, C15, C17, C18, C20, C21, C23, C24, C26, C27, C29, C3, C30, C32, C33, C35, C36, C38, C39, C41, C42, C44, C45, C47, C48, C5, C6, C8, C9, C? (x6): 10n, Capacitors_SMD:C_0805_HandSoldering, symbol C_Small
- added C51, C54, C69: 1µ, Capacitors_SMD:C_0805_HandSoldering, symbol C_Small
- added C52, C53: 100n, Capacitors_SMD:C_0805_HandSoldering, symbol C_Small
- added C55: 120p, Capacitors_SMD:C_0805_HandSoldering, symbol C_Small
- added C56, C58, C60, C64, C66, C68: 1n, Capacitors_SMD:C_0805_HandSoldering, symbol C_Small
- added C57: 200p, Capacitors_SMD:C_0805_HandSoldering, symbol C_Small
- added C59, C65, C67: 100p, Capacitors_SMD:C_0805_HandSoldering, symbol C_Small
- added C61: 50n, Capacitors_SMD:C_0805_HandSoldering, symbol C_Small
- added C62: 250µ, Capacitors_SMD:c_elec_8x5.4, symbol CP1_Small
- added C63: 10p, Capacitors_SMD:C_0805_HandSoldering, symbol C_Small
- added C? (x2): 47µ, Capacitors_SMD:C_1206_HandSoldering, symbol CP_Small
- added P4, P5, P6, P7: CONN_02X13, Socket_Strips:Socket_Strip_Straight_2x13, symbol CONN_02X13
- added P8: CONN_01X02, Socket_Strips:Socket_Strip_Angled_1x02, symbol CONN_01X02
- added R1: 1k, Resistors_SMD:R_0805_HandSoldering, symbol R
- added R10, R12, R4, R5, R7, R8, R9: 10k, Resistors_SMD:R_0805_HandSoldering, symbol R
- added R11, R13, R14, R2, R3, R6: 5k, Resistors_SMD:R_0805_HandSoldering, symbol R
- added R15, R16: 38.3k, Resistors_SMD:R_0805_HandSoldering, symbol R
- added R17: 7.5k, Resistors_SMD:R_0805_HandSoldering, symbol R
- added R18: 133k, Resistors_SMD:R_0805_HandSoldering, symbol R
- added R19: 5.36k, Resistors_SMD:R_0805_HandSoldering, symbol R
- added R20: 187k, Resistors_SMD:R_0805_HandSoldering, symbol R
- added R21: 10, Resistors_SMD:R_0805_HandSoldering, symbol R
- added RV1: 10k, Potentiometers:Potentiometer_WirePads_Small, symbol POT
- added unit 4 of U1
- added U10, U9: SST39SF020, Sockets_DIP:DIP-32__600, symbol SST39SF020
- added U11, U23: 74LS541, Sockets_DIP:DIP-20__300, symbol 74LS541
- added U13, U5, U6: 4040, Sockets_DIP:DIP-16__300, symbol 4040
- added U15: 74LS02, Sockets_DIP:DIP-14__300, symbol 74LS02
- added U17: 74LS32, Sockets_DIP:DIP-14__300, symbol 74LS32
- added U18, U32: DAC08, Sockets_DIP:DIP-16__300, symbol DAC08
- added U19: MCP1541-I/TO, Housings_TO-92:TO-92_Inline_Wide, symbol LM1084IS-3.3/NOPB
- added U20, U8: 74LS373, Sockets_DIP:DIP-20__300, symbol 74LS373
- added U21: 74HC138, Sockets_DIP:DIP-16__300, symbol 74LS138
- added U22, U33: TL074, Sockets_DIP:DIP-14__300, symbol TL074
- added U25: 74LS163, Sockets_DIP:DIP-16__300, symbol 74LS163
- added U28, U30: 74LS21, Sockets_DIP:DIP-14__300, symbol 74LS21
- added U34: LM386, Sockets_DIP:DIP-8__300, symbol LM386
- C2: renamed from C223; value 1µ -> 10n
- P2: renamed from P1; value 32kHz osc -> 1MHz osc
- P3: renamed from P?; footprint (none) -> Sockets_DIP:DIP-18__300
- U12: renamed from U?; footprint (none) -> Sockets_DIP:DIP-40__600
- U2, U27: renamed from U?; footprint (none) -> Sockets_DIP:DIP-14__300
- gave numbers to parts that had none: 2
- renumbered C203 to C1, C206 to C10, C207 to C13, C208 to C16, C209 to C19, C210 to C22, C211 to C25, C212 to C28, C213 to C31, C214 to C34, C215 to C37, C204 to C4, C216 to C40, C217 to C43, C218 to C46, C201 to C49, C202 to C50, C205 to C7, P3 to P1, U122 to U1, U4 to U14, U148 to U16, U124 to U24, U128 to U26, U134 to U3, U131 to U31, U133 to U4, U138 to U7
Connections:
- net labels added: 4.096V, Clk_gme_data, GM_adress_latch, GW0, GW1, GW2, GW3, GmSelectB0, GmSelectB1, Gm_db0, Gm_db1, Gm_db10, Gm_db11, Gm_db12, Gm_db13, Gm_db14, Gm_db15, Gm_db2, Gm_db3, Gm_db4, Gm_db5, Gm_db6, Gm_db7, Gm_db8, Gm_db9, Gm_pulse, Gwn, Maout, RST_GM0, RST_GM1, RST_GM2, RST_GM3, Tmr_rst, Vaout, Vrst, lGm_db0, lGm_db1, lGm_db10, lGm_db11, lGm_db12, lGm_db13, lGm_db14, lGm_db15, lGm_db2, lGm_db3, lGm_db4, lGm_db5, lGm_db6, lGm_db7, lGm_db8, lGm_db9
- net labels removed: A0_aud_v, A1_aud_v, A2_aud_v, A3_aud_v, Clk_main1, Voice_select0, Voice_select1, Voice_select2
- wire segments 308 -> 694
- no-connect marks 41 -> 80
Other:
- moved on the sheet: C49, C50, P3, U14, U16, U27B, U29, U2B
