File: Hardware/Digital board/Digital_board.sch (KiCad schematic (older format))
At the start: 141 parts, among them P1 CONN_01X04, P2 1MHz osc, P3 DIL18, P4 CONN_02X13, P5 CONN_02X13, P6 CONN_02X13, P7 CONN_02X13, P8 CONN_01X02, U1 74LS32, U10 SST39SF020, U11 74LS541, U12 Dip-mem_2Mx8b, U13 4040, U14 74LS541, U15 74LS02, U16 74LS373, U17 74LS32, U18 DAC08, U19 MCP1541-I/TO, U2 74LS21, U20 74LS373, U21 74HC138, U22 TL074, U23 74LS541, U24 4040, U25 74LS163, U26 SST39SF020, U27 74LS21, U28 74LS21, U29 74LS373, U3 4040, U30 74LS21, U31 4040, U32 DAC08, U33 TL074, U34 LM386, U4 4040, U5 4040, U6 4040, U7 74LS08, U8 74LS373, U9 SST39SF020

Commit message: Pcb design
Parts:
- removed C31, C34, C37, C40, C43, C46: 1µ, Capacitors_SMD:C_0805_HandSoldering, symbol C_Small
- removed C32, C33, C35, C36, C38, C39, C41, C42, C44, C45, C47, C48: 10n, Capacitors_SMD:C_0805_HandSoldering, symbol C_Small
- C49: footprint Capacitors_SMD:C_1206_HandSoldering -> Capacitors_SMD:c_elec_6.3x5.8
- C50: footprint Capacitors_SMD:C_1206_HandSoldering -> Capacitors_SMD:c_elec_6.3x5.7
- C57: value 200p -> 100p
- C70, C71: renamed from C?; footprint Capacitors_SMD:C_1206_HandSoldering -> Capacitors_SMD:c_elec_6.3x5.8
- gave numbers to parts that had none: 6
- renumbered U30 to U28
Other:
- moved on the sheet: U17A, U1D
