File: Hardware/Digital board/Digital_board.kicad_pcb (KiCad board)
At the start: 4 copper layers, 557 parts, among them P1 1.8MHz osc, P2 SW_DIP9, P3 CONN_01X04, P4 CONN_02X32, P5 CONN_02X20, P6 CONN_01X03, P7 CONN_02X05, U1 74HCT02, U10 74LS688, U100 74LS373, U101 74LS688, U102 74LS688, U103 74LS688, U104 74LS688, U105 4040, U106 4040, U107 4040, U108 4040, U109 74HCT02, U11 74LS688, U110 74LS688, U111 74LS688, U112 4040, U113 4040, U114 74LS688, U115 74LS688, U116 4040, U117 4040, U118 74LS373, U119 74LS373, U12 4040, U120 74LS373, U121 74LS373, U122 74LS32, U123 4040, U124 4040, U125 74LS541, U126 74LS541, U127 SST39SF020, U128 SST39SF020, U129 74LS30, U13 4040, U130 74LS30, U131 4040, U132 SST39SF020, U133 4040, U134 4040, U135 74LS688, U136 74HCT02, U137 4040, U138 74LS08, U139 4040, U14 4040, U140 74LS688, U141 74LS688, U142 74LS238, U143 74LS373, U144 74LS373, U145 74LS238, U146 74LS373, U147 74LS373, U148 74LS373, U149 4040, U15 4040, U150 74LS688, U151 4040, U152 74LS688, U153 4040, U154 74LS688, U155 74HCT02, U156 4040, U157 4040, U158 74LS688, U159 74LS688, U16 74LS541, U160 4040, U161 74LS373, U162 74LS688, U163 74LS373, U164 74LS373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

Commit message: Schematic ERC corrections
Parts:
- removed C100, C101, C102, C103, C104, C105, C106, C107, C108, C109, C110, C111, C112, C113, C114, C115, C116, C117, C118, C119, C120, C121, C122, C123, C124, C125, C126, C127, C128, C129, C130, C131, C132, C133, C134, C135, C136, C137, C138, C139, C140, C141, C142, C143, C144, C145, C146, C147, C148, C149, C150, C151, C152, C153, C154, C155, C156, C157, C158, C159, C160, C161, C162, C163, C164, C165, C166, C167, C168, C169, C170, C171, C172, C173, C174, C175, C176, C177, C178, C179, C180, C181, C182, C183, C184, C185, C186, C187, C188, C189, C190, C191, C192, C193, C194, C195, C196, C197, C198, C199, C200, C243, C244, C245, C246, C247, C248, C249, C250, C251, C252, C253, C254, C255, C256, C257, C258, C259, C260, C261, C262, C263, C264, C265, C266, C267, C268, C269, C270, C271, C272, C273, C274, C275, C276, C277, C278, C279, C280, C281, C282, C283, C284, C285, C286, C287, C288, C289, C290, C291, C292, C293, C294, C295, C296, C297, C298, C299, C300, C301, C302, C78, C79, C80, C81, C82, C83, C84, C85, C86, C87, C88, C89, C90, C91, C92, C93, C94, C95, C96, C97, C98, C99: 22n, Capacitors_SMD:C_0603_HandSoldering
- removed C201, C202: 47µ, Capacitors_SMD:C_1206_HandSoldering
- removed C203, C204, C205, C206, C207, C208, C209, C210, C211, C212, C213, C214, C215, C216, C217, C218, C219, C220, C221, C222, C223, C224, C225, C226, C227, C228, C229, C230, C231, C232, C233, C234, C235, C236, C237, C238, C239, C240, C241, C242: 1µ, Capacitors_SMD:C_0805_HandSoldering
- removed R24, R25: 100k, Resistors_SMD:R_0805_HandSoldering
- removed U100, U118, U119, U120, U121, U143, U144, U146, U147, U148, U161, U163, U164, U165, U166, U167, U168, U176, U193, U194, U195, U200, U203, U205, U206, U207, U209, U211, U233, U234, U235, U237, U239, U243, U244, U35, U40, U41, U42, U43, U45, U62, U66, U67, U68, U69, U72, U73, U74, U75, U93, U94, U95, U96, U97, U98, U99: 74LS373, Sockets_DIP:DIP-20__300
- removed U101, U102, U103, U104, U110, U111, U114, U115, U135, U140, U141, U150, U152, U154, U158, U159, U162, U171, U173, U175, U178, U185, U187, U188, U190, U196, U201, U214, U215, U217, U221, U223, U224, U225, U229, U230, U231, U236, U242, U47, U48, U49, U50, U56, U57, U60, U61, U70, U76, U77, U78, U79, U85, U86, U89, U90: 74LS688, Sockets_DIP:DIP-20__300
- removed U105, U106, U107, U108, U112, U113, U116, U117, U123, U124, U131, U133, U134, U137, U139, U149, U151, U153, U156, U157, U160, U169, U172, U174, U177, U182, U183, U184, U186, U192, U198, U212, U213, U216, U220, U222, U226, U227, U228, U232, U238, U240, U241, U51, U52, U53, U54, U58, U59, U63, U64, U65, U71, U80, U81, U82, U83, U87, U88, U91, U92: 4040, Sockets_DIP:DIP-16__300
- removed U109, U136, U155, U180, U219, U55, U84: 74HCT02, Sockets_DIP:DIP-14__300
- removed U122: 74LS32, Sockets_DIP:DIP-14__300
- removed U125, U126: 74LS541, Sockets_DIP:DIP-20__300
- removed U127, U128, U132: SST39SF020, Sockets_DIP:DIP-32__600
- removed U129, U130: 74LS30, Sockets_DIP:DIP-14__300
- removed U138: 74LS08, Sockets_DIP:DIP-14__300
- removed U142, U145, U36, U37: 74LS238, Sockets_DIP:DIP-16__300
- removed U170, U179, U181, U189, U191, U197, U199, U202, U204, U208, U210, U218, U38, U39, U44, U46: 74HC74, Sockets_DIP:DIP-14__300
- added P8: CONN_01X02, Socket_Strips:Socket_Strip_Angled_1x02, F.Cu at (251.2, 28.6)
- added R10: 10k, Resistors_SMD:R_0805_HandSoldering, F.Cu at (237.2, 149.7)
- added R11: 5k, Resistors_SMD:R_0805_HandSoldering, F.Cu at (279.0, 117.1)
- added R12: 10k, Resistors_SMD:R_0805_HandSoldering, F.Cu at (279.5, 110.8)
- added R13: 5k, Resistors_SMD:R_0805_HandSoldering, F.Cu at (257.8, 137.2)
- added R14: 5k, Resistors_SMD:R_0805_HandSoldering, F.Cu at (266.4, 127.8)
- added R15: 38.3k, Resistors_SMD:R_0805_HandSoldering, F.Cu at (284.8, 110.8)
- added R16: 38.3k, Resistors_SMD:R_0805_HandSoldering, F.Cu at (290.0, 104.6)
- added R17: 7.5k, Resistors_SMD:R_0805_HandSoldering, F.Cu at (276.7, 123.4)
- added R18: 133k, Resistors_SMD:R_0805_HandSoldering, F.Cu at (290.0, 110.9)
- added R19: 5.36k, Resistors_SMD:R_0805_HandSoldering, F.Cu at (284.3, 117.1)
- added R20: 187k, Resistors_SMD:R_0805_HandSoldering, F.Cu at (263.0, 134.1)
- added R21: 10, Resistors_SMD:R_0805_HandSoldering, F.Cu at (252.7, 143.5)
- added R3: 5k, Resistors_SMD:R_0805_HandSoldering, F.Cu at (261.2, 127.8)
- added R4: 10k, Resistors_SMD:R_0805_HandSoldering, F.Cu at (273.8, 114.0)
- added R5: 10k, Resistors_SMD:R_0805_HandSoldering, F.Cu at (284.6, 104.5)
- added R6: 5k, Resistors_SMD:R_0805_HandSoldering, F.Cu at (252.5, 137.2)
- added R7: 10k, Resistors_SMD:R_0805_HandSoldering, F.Cu at (271.5, 120.3)
- added R8: 10k, Resistors_SMD:R_0805_HandSoldering, F.Cu at (292.7, 98.3)
- added R9: 10k, Resistors_SMD:R_0805_HandSoldering, F.Cu at (242.4, 146.6)
- added RV1: 10k, Potentiometers:Potentiometer_WirePads_Small, F.Cu at (286.4, 64.4)
- C1, C10, C13, C16, C19, C22, C25, C28, C31, C34, C37, C4, C40, C43, C46, C51, C54, C69, C7: value 22n -> 1µ; footprint Capacitors_SMD:C_0603_HandSoldering -> Capacitors_SMD:C_0805_HandSoldering
- C11, C12, C14, C15, C17, C18, C2, C20, C21, C23, C24, C26, C27, C29, C3, C30, C32, C33, C35, C36, C38, C39, C41, C42, C44, C45, C47, C48, C5, C6, C72, C73, C74, C75, C76, C77, C8, C9: value 22n -> 10n; footprint Capacitors_SMD:C_0603_HandSoldering -> Capacitors_SMD:C_0805_HandSoldering
- C49, C70, C71: value 22n -> 47µ; footprint Capacitors_SMD:C_0603_HandSoldering -> Capacitors_SMD:c_elec_6.3x5.8
- C50: value 22n -> 47µ; footprint Capacitors_SMD:C_0603_HandSoldering -> Capacitors_SMD:c_elec_6.3x5.7
- C52, C53: value 22n -> 100n; footprint Capacitors_SMD:C_0603_HandSoldering -> Capacitors_SMD:C_0805_HandSoldering
- C55: value 22n -> 120p; footprint Capacitors_SMD:C_0603_HandSoldering -> Capacitors_SMD:C_0805_HandSoldering
- C56, C58, C60, C64, C66, C68: value 22n -> 1n; footprint Capacitors_SMD:C_0603_HandSoldering -> Capacitors_SMD:C_0805_HandSoldering
- C57: value 22n -> 200p; footprint Capacitors_SMD:C_0603_HandSoldering -> Capacitors_SMD:C_0805_HandSoldering
- C59, C65, C67: value 22n -> 100p; footprint Capacitors_SMD:C_0603_HandSoldering -> Capacitors_SMD:C_0805_HandSoldering
- C61: value 22n -> 50n; footprint Capacitors_SMD:C_0603_HandSoldering -> Capacitors_SMD:C_0805_HandSoldering
- C62: value 22n -> 250µ; footprint Capacitors_SMD:C_0603_HandSoldering -> Capacitors_SMD:c_elec_8x5.4
- C63: value 22n -> 10p; footprint Capacitors_SMD:C_0603_HandSoldering -> Capacitors_SMD:C_0805_HandSoldering
- P1: value 1.8MHz osc -> CONN_01X04; footprint Sockets_DIP:DIP-14__300 -> Socket_Strips:Socket_Strip_Straight_1x04
- P2: value SW_DIP9 -> 1MHz osc; footprint Sockets_DIP:DIP-18__300 -> Sockets_DIP:DIP-14__300
- P3: value CONN_01X04 -> DIL18; footprint Socket_Strips:Socket_Strip_Straight_1x04 -> Sockets_DIP:DIP-18__300
- P4: value CONN_02X32 -> CONN_02X13; footprint Socket_Strips:Socket_Strip_Straight_2x32 -> Socket_Strips:Socket_Strip_Straight_2x13
- P5: value CONN_02X20 -> CONN_02X13; footprint Socket_Strips:Socket_Strip_Straight_2x20 -> Socket_Strips:Socket_Strip_Straight_2x13
- P6: value CONN_01X03 -> CONN_02X13; footprint Socket_Strips:Socket_Strip_Straight_1x03 -> Socket_Strips:Socket_Strip_Straight_2x13
- P7: value CONN_02X05 -> CONN_02X13; footprint Socket_Strips:Socket_Strip_Straight_2x05 -> Socket_Strips:Socket_Strip_Straight_2x13
- R1: value 100k -> 1k
- R2: value 100k -> 5k
- U1: value 74HCT02 -> 74LS32
- U10, U9: value 74LS688 -> SST39SF020; footprint Sockets_DIP:DIP-20__300 -> Sockets_DIP:DIP-32__600
- U11, U23: value 74LS688 -> 74LS541
- U12: value 4040 -> Dip-mem_2Mx8b; footprint Sockets_DIP:DIP-16__300 -> Sockets_DIP:DIP-40__600
- U14: value 4040 -> 74LS541; footprint Sockets_DIP:DIP-16__300 -> Sockets_DIP:DIP-20__300
- U15: value 4040 -> 74LS02; footprint Sockets_DIP:DIP-16__300 -> Sockets_DIP:DIP-14__300
- U16: value 74LS541 -> 74LS373
- U17: value 74LS541 -> 74LS32; footprint Sockets_DIP:DIP-20__300 -> Sockets_DIP:DIP-14__300; moved to F.Cu
- U18: value SST39SF020 -> DAC08; footprint Sockets_DIP:DIP-32__600 -> Sockets_DIP:DIP-16__300; moved to F.Cu
- U19: value SST39SF020 -> MCP1541-I/TO; footprint Sockets_DIP:DIP-32__600 -> Housings_TO-92:TO-92_Inline_Wide
- U2: value 74LS373 -> 74LS21; footprint Sockets_DIP:DIP-20__300 -> Sockets_DIP:DIP-14__300
- U20: value 74LS30 -> 74LS373; footprint Sockets_DIP:DIP-14__300 -> Sockets_DIP:DIP-20__300
- U21: value 74LS30 -> 74HC138; footprint Sockets_DIP:DIP-14__300 -> Sockets_DIP:DIP-16__300; moved to F.Cu
- U22: value 74HCT02 -> TL074
- U24: value 74LS688 -> 4040; footprint Sockets_DIP:DIP-20__300 -> Sockets_DIP:DIP-16__300
- U25: value 4040 -> 74LS163
- U26: value 4040 -> SST39SF020; footprint Sockets_DIP:DIP-16__300 -> Sockets_DIP:DIP-32__600
- U27, U28: value 74LS688 -> 74LS21; footprint Sockets_DIP:DIP-20__300 -> Sockets_DIP:DIP-14__300
- U29: value 4040 -> 74LS373; footprint Sockets_DIP:DIP-16__300 -> Sockets_DIP:DIP-20__300
- U3, U5, U6: value 74LS373 -> 4040; footprint Sockets_DIP:DIP-20__300 -> Sockets_DIP:DIP-16__300
- U30: value 4040 -> 74LS21; footprint Sockets_DIP:DIP-16__300 -> Sockets_DIP:DIP-14__300
- U31: moved to F.Cu
- U32: value 74LS373 -> DAC08; footprint Sockets_DIP:DIP-20__300 -> Sockets_DIP:DIP-16__300
- U33: value 74LS373 -> TL074; footprint Sockets_DIP:DIP-20__300 -> Sockets_DIP:DIP-14__300
- U34: value 74LS373 -> LM386; footprint Sockets_DIP:DIP-20__300 -> Sockets_DIP:DIP-8__300
- U4: value 74LS541 -> 4040; footprint Sockets_DIP:DIP-20__300 -> Sockets_DIP:DIP-16__300
- U7: value 4040 -> 74LS08; footprint Sockets_DIP:DIP-16__300 -> Sockets_DIP:DIP-14__300
- U8: value 74LS688 -> 74LS373
- moved C70 687.4 mm to (21.8, 81.5)
- moved C74 678.5 mm to (25.5, 67.7)
- moved C77 654.0 mm to (36.0, 68.1)
- moved C71 646.7 mm to (43.2, 58.8)
- moved C76 644.3 mm to (31.8, 73.3)
- moved C73 641.1 mm to (34.0, 80.2)
- moved C75 629.3 mm to (41.5, 74.9)
- moved C72 626.2 mm to (49.0, 71.4)
- moved C60 545.0 mm to (165.9, 149.3)
- moved C59 536.5 mm to (155.8, 149.3)
- moved U12 533.1 mm to (79.1, 46.0)
- moved C61 531.6 mm to (171.0, 149.3)
- moved C58 529.3 mm to (160.9, 149.3)
- moved C57 519.1 mm to (181.1, 149.3)
- moved C36 506.0 mm to (176.0, 149.3)
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Connections:
- C51 pad 1: VCC -> GND
- C51 pad 2: GND -> Net-(C51-Pad2)
- C52 pad 1: VCC -> Net-(C52-Pad1)
- C52 pad 2: GND -> -12VA
- C53 pad 1: VCC -> Net-(C53-Pad1)
- C53 pad 2: GND -> -12VA
- C54 pad 1: VCC -> Net-(C54-Pad1)
- C54 pad 2: GND -> Net-(C54-Pad2)
- C55 pad 1: VCC -> Net-(C55-Pad1)
- C56 pad 1: VCC -> Net-(C56-Pad1)
- C56 pad 2: GND -> Net-(C56-Pad2)
- C57 pad 1: VCC -> Net-(C57-Pad1)
- C58 pad 1: VCC -> Net-(C58-Pad1)
- C58 pad 2: GND -> Net-(C58-Pad2)
- C59 pad 1: VCC -> Net-(C59-Pad1)
- C60 pad 1: VCC -> Net-(C60-Pad1)
- C60 pad 2: GND -> Net-(C60-Pad2)
- C61 pad 1: VCC -> Net-(C61-Pad1)
- C61 pad 2: GND -> Net-(C61-Pad2)
- C62 pad 1: VCC -> Net-(C61-Pad1)
- C62 pad 2: GND -> Net-(C62-Pad2)
- C63 pad 1: VCC -> Net-(C55-Pad1)
- C64 pad 1: VCC -> Net-(C56-Pad1)
- C64 pad 2: GND -> Net-(C56-Pad2)
- C65 pad 1: VCC -> Net-(C57-Pad1)
- C66 pad 1: VCC -> Net-(C58-Pad1)
- C66 pad 2: GND -> Net-(C58-Pad2)
- C67 pad 1: VCC -> Net-(C59-Pad1)
- C68 pad 1: VCC -> Net-(C60-Pad1)
- C68 pad 2: GND -> Net-(C60-Pad2)
- C69 pad 1: VCC -> GND
- C69 pad 2: GND -> (no net)
- C70 pad 1: VCC -> +12VA
- C71 pad 1: VCC -> GND
- C71 pad 2: GND -> -12VA
- C72 pad 1: VCC -> +12VA
- C73 pad 1: VCC -> GND
- C73 pad 2: GND -> -12VA
- C74 pad 1: VCC -> +12VA
- C75 pad 1: VCC -> GND
- C75 pad 2: GND -> -12VA
- C76 pad 1: VCC -> +12VA
- C77 pad 1: VCC -> GND
- C77 pad 2: GND -> -12VA
- P1 pad 1: Net-(P1-Pad1) -> +12VA
- P1 pad 2: Net-(P1-Pad2) -> -12VA
- P1 pad 3: Net-(P1-Pad3) -> VCC
- P1 pad 4: Net-(P1-Pad4) -> GND
- P2 pad 1: VCC -> (no net)
- P2 pad 10: /BS9 -> (no net)
- P2 pad 11: /BS8 -> (no net)
- P2 pad 12: /BS7 -> (no net)
- P2 pad 13: /BS6 -> (no net)
- P2 pad 14: /BS5 -> Net-(P2-Pad14)
- P2 pad 2: VCC -> (no net)
- P2 pad 3: VCC -> (no net)
- P2 pad 4: VCC -> (no net)
- P2 pad 5: VCC -> (no net)
- P2 pad 6: VCC -> (no net)
- P2 pad 7: VCC -> GND
- P2 pad 9: VCC -> (no net)
- P3 pad 1: +12VA -> VCC
- P3 pad 2: -12VA -> VCC
- P3 pad 4: GND -> VCC
- P4 pad 1: /Av_amp0_C0 -> VCC
- P4 pad 10: /Av_amp0_C9 -> /RST_GM2
- P4 pad 11: /Av_amp1_C1 -> /lGm_db4
- P4 pad 12: /Av_amp1_C9 -> GND
- P4 pad 13: /Av_amp2_C1 -> /lGm_db5
- P4 pad 14: /Av_amp2_C9 -> /Clk_main6
- P4 pad 15: /Av_amp3_C1 -> /lGm_db6
- P4 pad 16: /Av_amp3_C9 -> GND
- P4 pad 17: /Av_amp0_C2 -> /lGm_db7
- P4 pad 18: /Av_amp0_C10 -> /GW2
- P4 pad 19: /Av_amp1_C2 -> /lGm_db8
- P4 pad 2: /Av_amp0_C8 -> /lGm_db12
- P4 pad 20: /Av_amp1_C10 -> GND
- P4 pad 21: /Av_amp2_C2 -> /lGm_db9
- P4 pad 22: /Av_amp2_C10 -> VCC
- P4 pad 23: /Av_amp3_C2 -> /lGm_db10
- P4 pad 24: /Av_amp3_C10 -> VCC
- P4 pad 25: /Av_amp0_C3 -> /lGm_db11
- P4 pad 26: /Av_amp0_C11 -> GND
- P4 pad 3: /Av_amp1_C0 -> /lGm_db0
- P4 pad 4: /Av_amp1_C8 -> /lGm_db13
- P4 pad 5: /Av_amp2_C0 -> /lGm_db1
- P4 pad 6: /Av_amp2_C8 -> /lGm_db14
- P4 pad 7: /Av_amp3_C0 -> /lGm_db2
- P4 pad 8: /Av_amp3_C8 -> /lGm_db15
- P4 pad 9: /Av_amp0_C1 -> /lGm_db3
- P5 pad 1: /Amout0 -> VCC
- P5 pad 10: /Avout0 -> /RST_GM0
- P5 pad 11: /Amout5 -> /lGm_db4
- P5 pad 12: /Avout1 -> GND
- P5 pad 13: /Amout6 -> /lGm_db5
- P5 pad 14: /Avout2 -> /Clk_main4
- P5 pad 15: /Amout7 -> /lGm_db6
- P5 pad 16: /Avout3 -> GND
- P5 pad 17: /Amout8 -> /lGm_db7
- P5 pad 18: /Avout4 -> /GW0
- P5 pad 19: /Amout9 -> /lGm_db8
- P5 pad 2: /AD_db4 -> /lGm_db12
- P5 pad 20: /Avout5 -> GND
- P5 pad 21: /Amout10 -> /lGm_db9
- P5 pad 22: /Avout6 -> VCC
- P5 pad 23: /Amout11 -> /lGm_db10
- P5 pad 24: /Avout7 -> VCC
- P5 pad 25: /Amout12 -> /lGm_db11
- P5 pad 26: /Avout8 -> GND
- P5 pad 3: /Amout1 -> /lGm_db0
- P5 pad 4: /AD_db5 -> /lGm_db13
- P5 pad 5: /Amout2 -> /lGm_db1
- P5 pad 6: /AD_db6 -> /lGm_db14
- P5 pad 7: /Amout3 -> /lGm_db2
- P5 pad 8: /AD_db7 -> /lGm_db15
- P5 pad 9: /Amout4 -> /lGm_db3
- P6 pad 1: Clk_main7 -> VCC
- P6 pad 2: Clk_main6 -> /lGm_db12
- P6 pad 3: GND -> /lGm_db0
- P7 pad 1: /Master_reset -> VCC
- P7 pad 10: Net-(P7-Pad10) -> /RST_GM1
- P7 pad 2: /Voice_reset_blank -> /lGm_db12
- P7 pad 3: /Voice_select0 -> /lGm_db0
- P7 pad 4: Net-(P7-Pad4) -> /lGm_db13
- P7 pad 5: /Voice_select1 -> /lGm_db1
- P7 pad 6: Net-(P7-Pad6) -> /lGm_db14
- P7 pad 7: /Voice_select2 -> /lGm_db2
- P7 pad 8: Net-(P7-Pad8) -> /lGm_db15
- P7 pad 9: Net-(P7-Pad9) -> /lGm_db3
- R1 pad 1: /BS1 -> Net-(C51-Pad2)
- R1 pad 2: GND -> VCC
- R2 pad 1: GND -> /4.096V
- R2 pad 2: /BS2 -> Net-(R2-Pad2)
- U1 pad 1: Net-(U1-Pad1) -> /Rst_audM
- U1 pad 10: Net-(U1-Pad10) -> /Rst_Gam
- U1 pad 11: GND -> /Rst_Gam
- U1 pad 12: GND -> /Gwn
- U1 pad 13: Net-(U1-Pad13) -> /Gm_pulse
- U1 pad 2: /Rst_aud_1 -> /Master_reset
- U1 pad 3: /Rst_aud_2 -> Net-(U1-Pad3)
- U1 pad 5: /Rst_audV_1 -> /Master_reset
- U1 pad 6: /Rst_audV_2 -> /Vrst
- U1 pad 8: GND -> Net-(U1-Pad4)
- U1 pad 9: GND -> Net-(U1-Pad9)
- U10 pad 1: GND -> (no net)
- U10 pad 10: GND -> Net-(U10-Pad10)
- U10 pad 11: Net-(U10-Pad11) -> /GmSelectB1
- U10 pad 12: Net-(U10-Pad12) -> /GmSelectB0
- U10 pad 13: Net-(U10-Pad13) -> /Gm_db0
- U10 pad 14: Net-(U10-Pad14) -> /Gm_db1
- U10 pad 15: Net-(U10-Pad15) -> /Gm_db2
- U10 pad 16: Net-(U10-Pad16) -> GND
- U10 pad 17: Net-(U10-Pad17) -> /Gm_db3
- U10 pad 18: Net-(U10-Pad18) -> /Gm_db4
- U10 pad 19: Net-(U10-Pad19) -> /Gm_db5
- U10 pad 20: VCC -> /Gm_db6
- U11 pad 11: Net-(U11-Pad11) -> /lGm_db7
- U11 pad 12: Net-(U11-Pad12) -> /lGm_db6
- U11 pad 13: Net-(U11-Pad13) -> /lGm_db5
- U11 pad 14: Net-(U11-Pad14) -> /lGm_db4
- U11 pad 15: Net-(U11-Pad15) -> /lGm_db3
- U11 pad 16: Net-(U11-Pad16) -> /lGm_db2
- U11 pad 17: Net-(U11-Pad17) -> /lGm_db1
- U11 pad 18: Net-(U11-Pad18) -> /lGm_db0
- U11 pad 19: Net-(U11-Pad19) -> GND
- U12 pad 1: Net-(U12-Pad1) -> VCC
- U12 pad 10: /Clk_main1 -> /Clk_divb8
- U12 pad 11: /Rst_clk_audm3 -> /Clk_divb9
- U12 pad 12: Net-(U12-Pad12) -> /Clk_divb10
- U12 pad 13: Net-(U12-Pad13) -> /Clk_divb11
- U12 pad 14: Net-(U12-Pad14) -> /Clk_divb12
- U12 pad 15: Net-(U12-Pad15) -> /Clk_divb13
- U12 pad 16: VCC -> /Clk_divb14
- U12 pad 2: Net-(U12-Pad2) -> /Clk_divb0
- U12 pad 3: Net-(U12-Pad3) -> /Clk_divb1
- U12 pad 4: Net-(U12-Pad4) -> /Clk_divb2
- U12 pad 5: Net-(U12-Pad5) -> /Clk_divb3
- U12 pad 6: Net-(U12-Pad6) -> /Clk_divb4
- U12 pad 7: Net-(U12-Pad7) -> /Clk_divb5
- U12 pad 8: GND -> /Clk_divb6
- U12 pad 9: Net-(U12-Pad9) -> /Clk_divb7
- U13 pad 1: Net-(U13-Pad1) -> (no net)
- U13 pad 10: /Clk_main1 -> /Clk_gme_data
- U13 pad 11: /Rst_clk_audm2 -> GND
- U13 pad 12: Net-(U13-Pad12) -> (no net)
- U13 pad 13: Net-(U13-Pad13) -> (no net)
- U13 pad 14: Net-(U13-Pad14) -> (no net)
- U13 pad 15: Net-(U13-Pad15) -> (no net)
- U13 pad 2: Net-(U13-Pad2) -> Net-(U10-Pad30)
- U13 pad 3: Net-(U13-Pad3) -> Net-(U10-Pad2)
- U13 pad 4: Net-(U13-Pad4) -> (no net)
- U13 pad 5: Net-(U13-Pad5) -> Net-(U10-Pad3)
- U13 pad 6: Net-(U13-Pad6) -> Net-(U10-Pad29)
- U13 pad 7: Net-(U13-Pad7) -> Net-(U10-Pad28)
- U13 pad 9: Net-(U13-Pad9) -> Net-(U10-Pad4)
- U14 pad 1: Net-(U14-Pad1) -> GND
- U14 pad 10: /Clk_main1 -> GND
- U14 pad 11: /Rst_clk_audm1 -> Net-(U14-Pad11)
- U14 pad 12: Net-(U14-Pad12) -> /Clk_main6
- U14 pad 13: Net-(U10-Pad18) -> /Clk_main5
- U14 pad 14: Net-(U14-Pad14) -> /Clk_main4
- U14 pad 15: Net-(U14-Pad15) -> /Clk_main3
- U14 pad 16: VCC -> /Clk_main2
- U14 pad 2: Net-(U10-Pad14) -> Net-(U14-Pad2)
- U14 pad 3: Net-(U10-Pad12) -> Net-(U14-Pad18)
- U14 pad 4: Net-(U10-Pad16) -> Net-(U14-Pad18)
- U14 pad 5: Net-(U10-Pad9) -> Net-(U14-Pad18)
- U14 pad 6: Net-(U10-Pad7) -> Net-(U14-Pad18)
- U14 pad 7: Net-(U10-Pad5) -> Net-(U14-Pad18)
- U14 pad 8: GND -> Net-(U14-Pad18)
- U14 pad 9: Net-(U10-Pad3) -> Net-(C51-Pad2)
- U15 pad 1: Net-(U15-Pad1) -> (no net)
- U15 pad 10: /Clk_main1 -> /Master_reset
- U15 pad 11: /Rst_clk_audm0 -> /Master_reset
- U15 pad 12: Net-(U15-Pad12) -> /Rst_Gam
- U15 pad 13: Net-(U11-Pad18) -> /GM_adress_latch
- U15 pad 14: Net-(U15-Pad14) -> VCC
- U15 pad 2: Net-(U11-Pad14) -> GND
- U15 pad 3: Net-(U11-Pad12) -> GND
- U15 pad 4: Net-(U11-Pad16) -> (no net)
- U15 pad 5: Net-(U11-Pad9) -> GND
- U15 pad 6: Net-(U11-Pad7) -> GND
- U15 pad 7: Net-(U11-Pad5) -> GND
- U15 pad 9: Net-(U11-Pad3) -> Net-(U14-Pad11)
- U16 pad 11: /AM_db15 -> /Clk_main3
- U16 pad 12: /AM_db14 -> Net-(U16-Pad12)
- U16 pad 13: /AM_db13 -> /AV_db4
- U16 pad 14: /AM_db12 -> /AV_db5
- U16 pad 15: /AM_db11 -> Net-(U16-Pad15)
- U16 pad 16: /AM_db10 -> Net-(U16-Pad16)
- U16 pad 17: /AM_db9 -> /AV_db6
- U16 pad 18: /AM_db8 -> /AV_db7
- U16 pad 19: GND -> Net-(U16-Pad19)
- U16 pad 3: Net-(U16-Pad3) -> /AV_db0
- U16 pad 4: Net-(U16-Pad4) -> /AV_db1
- U16 pad 7: Net-(U16-Pad7) -> /AV_db2
- U16 pad 8: Net-(U16-Pad8) -> /AV_db3
- U17 pad 10: GND -> Net-(U17-Pad10)
- U17 pad 11: /AM_db7 -> Net-(U17-Pad11)
- U17 pad 12: /AM_db6 -> /GW3
- U17 pad 13: /AM_db5 -> /GW2
- U17 pad 14: /AM_db4 -> VCC
- U17 pad 2: Net-(U17-Pad2) -> GND
- U17 pad 3: Net-(U17-Pad3) -> (no net)
- U17 pad 4: Net-(U17-Pad4) -> /GW1
- U17 pad 5: Net-(U17-Pad5) -> /GW0
- U17 pad 6: Net-(U17-Pad6) -> Net-(U17-Pad10)
- U17 pad 7: Net-(U17-Pad7) -> GND
- U17 pad 8: Net-(U17-Pad8) -> /Gwn
- U17 pad 9: Net-(U17-Pad9) -> Net-(U17-Pad11)
- U18 pad 1: Net-(U18-Pad1) -> (no net)
- U18 pad 10: Net-(U18-Pad10) -> Net-(U16-Pad15)
- U18 pad 11: Net-(U18-Pad11) -> Net-(U16-Pad16)
- U18 pad 12: Net-(U18-Pad12) -> Net-(U16-Pad19)
- U18 pad 13: Net-(U16-Pad2) -> VCC
- U18 pad 14: Net-(U16-Pad3) -> Net-(R3-Pad2)
- U18 pad 15: Net-(U16-Pad4) -> GND
- U18 pad 16: GND -> Net-(C52-Pad1)
- U18 pad 2: /BS1 -> Net-(R2-Pad2)
- U18 pad 3: /A3_aud_m -> -12VA
- U18 pad 4: /A0_aud_m -> Net-(R6-Pad2)
- U18 pad 5: Net-(U18-Pad5) -> Net-(U16-Pad2)
- U18 pad 6: Net-(U18-Pad6) -> Net-(U16-Pad5)
- U18 pad 7: Net-(U18-Pad7) -> Net-(U16-Pad6)
- U18 pad 8: Net-(U18-Pad8) -> Net-(U16-Pad9)
- U18 pad 9: Net-(U18-Pad9) -> Net-(U16-Pad12)
- U19 pad 1: Net-(U19-Pad1) -> GND
- U19 pad 2: /BS1 -> Net-(U19-Pad2)
- U19 pad 3: /A3_aud_m -> +12VA
- U2 pad 1: GND -> /AM_db0
- U2 pad 10: GND -> /AM_db5
- U2 pad 11: /Chm_3 -> (no net)
- U2 pad 12: Net-(U2-Pad12) -> /AM_db6
- U2 pad 13: /AM_db4 -> /AM_db7
- U2 pad 14: /AM_db5 -> VCC
- U2 pad 2: Net-(U2-Pad2) -> /AM_db1
- U2 pad 3: /AM_db0 -> (no net)
- U2 pad 4: /AM_db1 -> /AM_db2
- U2 pad 5: Net-(U2-Pad5) -> /AM_db3
- U2 pad 7: /AM_db2 -> GND
- U2 pad 8: /AM_db3 -> Net-(U2-Pad8)
- U2 pad 9: Net-(U2-Pad9) -> /AM_db4
- U20 pad 1: Net-(U16-Pad2) -> GND
- U20 pad 10: (no net) -> GND
- U20 pad 11: Net-(U16-Pad8) -> /GM_adress_latch
- U20 pad 12: Net-(U16-Pad9) -> Net-(U20-Pad12)
- U20 pad 13: (no net) -> /Gm_db12
- U20 pad 14: VCC -> /Gm_db13
- U20 pad 2: Net-(U16-Pad3) -> Net-(U20-Pad2)
- U20 pad 3: Net-(U16-Pad4) -> /Gm_db8
- U20 pad 4: Net-(U16-Pad5) -> /Gm_db9
- U20 pad 5: Net-(U16-Pad6) -> Net-(U20-Pad5)
- U20 pad 6: Net-(U16-Pad7) -> Net-(U20-Pad6)
- U20 pad 7: GND -> /Gm_db10
- U20 pad 8: /Rst_aud_1 -> /Gm_db11
- U20 pad 9: (no net) -> Net-(U20-Pad9)
- U21 pad 1: Net-(U17-Pad9) -> /GmSelectB0
- U21 pad 11: Net-(U17-Pad3) -> (no net)
- U21 pad 12: Net-(U17-Pad2) -> /RST_GM3
- U21 pad 13: (no net) -> /RST_GM2
- U21 pad 14: VCC -> /RST_GM1
- U21 pad 2: Net-(U17-Pad8) -> /GmSelectB1
- U21 pad 3: Net-(U17-Pad7) -> GND
- U21 pad 4: Net-(U17-Pad6) -> /GM_adress_latch
- U21 pad 5: Net-(U17-Pad5) -> /Master_reset
- U21 pad 6: Net-(U17-Pad4) -> VCC
- U21 pad 7: GND -> (no net)
- U21 pad 8: /Rst_aud_2 -> GND
- U22 pad 1: /Rst_clk_audm3 -> /4.096V
- U22 pad 10: /Rst_clk_audm1 -> GND
- U22 pad 11: Net-(U11-Pad19) -> -12VA
- U22 pad 12: Net-(U22-Pad12) -> Net-(C54-Pad1)
- U22 pad 13: /Rst_clk_audm0 -> Net-(R15-Pad2)
- U22 pad 14: VCC -> Net-(R15-Pad2)
- U22 pad 2: Net-(U22-Pad2) -> /4.096V
- U22 pad 3: Net-(U22-Pad3) -> Net-(U19-Pad2)
- U22 pad 4: /Rst_clk_audm2 -> +12VA
- U22 pad 5: Net-(U22-Pad5) -> GND
- U22 pad 6: Net-(U22-Pad6) -> Net-(R6-Pad2)
- U22 pad 7: GND -> /Vaout
- U22 pad 8: Net-(U10-Pad19) -> Net-(C54-Pad2)
- U22 pad 9: Net-(U22-Pad9) -> Net-(R10-Pad1)
- U23 pad 11: Net-(U23-Pad11) -> /lGm_db15
- U23 pad 12: Net-(U23-Pad12) -> /lGm_db14
- U23 pad 13: Net-(U23-Pad13) -> /lGm_db13
- U23 pad 14: Net-(U23-Pad14) -> /lGm_db12
- U23 pad 15: Net-(U23-Pad15) -> /lGm_db11
- U23 pad 16: Net-(U23-Pad16) -> /lGm_db10
- U23 pad 17: Net-(U23-Pad17) -> /lGm_db9
- U23 pad 18: Net-(U23-Pad18) -> /lGm_db8
- U23 pad 19: Net-(U22-Pad3) -> GND
- U23 pad 2: Net-(U12-Pad12) -> Net-(U20-Pad2)
- U23 pad 3: Net-(U23-Pad3) -> Net-(U20-Pad5)
- U23 pad 4: Net-(U12-Pad14) -> Net-(U20-Pad6)
- U23 pad 5: Net-(U23-Pad5) -> Net-(U20-Pad9)
- U23 pad 6: Net-(U12-Pad15) -> Net-(U20-Pad12)
- U23 pad 7: Net-(U23-Pad7) -> Net-(U20-Pad15)
- U23 pad 8: Net-(U12-Pad1) -> Net-(U20-Pad16)
- U23 pad 9: Net-(U23-Pad9) -> Net-(U20-Pad19)
- U24 pad 1: GND -> /Clk_audv_data
- U24 pad 10: GND -> /Clk_main3
- U24 pad 11: Net-(U24-Pad11) -> /Vrst
- U24 pad 16: Net-(U24-Pad16) -> VCC
- U24 pad 2: Net-(U13-Pad12) -> Net-(U24-Pad2)
- U24 pad 4: Net-(U13-Pad14) -> Net-(U24-Pad4)
- U24 pad 6: Net-(U13-Pad15) -> Net-(U24-Pad6)
- U24 pad 8: Net-(U13-Pad1) -> GND
- U25 pad 1: Net-(U25-Pad1) -> VCC
- U25 pad 10: Net-(U12-Pad1) -> VCC
- U25 pad 11: /Rst_clk_audm3 -> Net-(U25-Pad11)
- U25 pad 15: Net-(U25-Pad15) -> (no net)
- U25 pad 2: Net-(U25-Pad2) -> /Clk_divb14
- U25 pad 3: Net-(U25-Pad3) -> Net-(P3-Pad15)
- U25 pad 4: Net-(U25-Pad4) -> Net-(P3-Pad16)
- U25 pad 5: Net-(U23-Pad17) -> Net-(P3-Pad17)
- U25 pad 6: Net-(U23-Pad15) -> Net-(P3-Pad18)
- U25 pad 7: Net-(U23-Pad13) -> VCC
- U25 pad 9: Net-(U23-Pad11) -> /GM_adress_latch
- U26 pad 1: Net-(U26-Pad1) -> (no net)
- U26 pad 10: Net-(U13-Pad1) -> Net-(U24-Pad6)
- U26 pad 11: /Rst_clk_audm2 -> Net-(U24-Pad7)
- U26 pad 12: Net-(U26-Pad12) -> Net-(U24-Pad9)
- U26 pad 13: Net-(U26-Pad13) -> /AV_db0
- U26 pad 14: Net-(U26-Pad14) -> /AV_db1
- U26 pad 15: Net-(U26-Pad15) -> /AV_db2
- U26 pad 16: VCC -> GND
- U26 pad 5: Net-(U24-Pad17) -> Net-(U24-Pad13)
- U26 pad 6: Net-(U24-Pad15) -> Net-(U24-Pad4)
- U26 pad 7: Net-(U24-Pad13) -> Net-(U24-Pad2)
- U26 pad 8: GND -> Net-(U24-Pad3)
- U26 pad 9: Net-(U24-Pad11) -> Net-(U24-Pad5)
- U27 pad 1: GND -> /AV_db7
- U27 pad 10: GND -> /AV_db2
- U27 pad 11: Net-(U27-Pad11) -> (no net)
- U27 pad 12: Net-(U27-Pad12) -> /AV_db1
- U27 pad 13: Net-(U27-Pad13) -> /AV_db0
- U27 pad 14: Net-(U27-Pad14) -> VCC
- U27 pad 2: Net-(U14-Pad12) -> /AV_db6
- U27 pad 3: Net-(U27-Pad3) -> (no net)
- U27 pad 4: Net-(U14-Pad14) -> /AV_db5
- U27 pad 5: Net-(U27-Pad5) -> /AV_db4
- U27 pad 6: Net-(U14-Pad15) -> Net-(U27-Pad6)
- U27 pad 7: Net-(U27-Pad7) -> GND
- U27 pad 8: Net-(U14-Pad1) -> Net-(U27-Pad8)
- U27 pad 9: Net-(U27-Pad9) -> /AV_db3
- U28 pad 1: GND -> Net-(U25-Pad14)
- U28 pad 10: GND -> (no net)
- U28 pad 11: Net-(U28-Pad11) -> (no net)
- U28 pad 12: Net-(U28-Pad12) -> (no net)
- U28 pad 13: Net-(U28-Pad13) -> (no net)
- U28 pad 14: Net-(U28-Pad14) -> VCC
- U28 pad 2: Net-(U15-Pad12) -> Net-(U25-Pad13)
- U28 pad 3: Net-(U28-Pad3) -> (no net)
- U28 pad 4: Net-(U15-Pad14) -> Net-(U25-Pad12)
- U28 pad 5: Net-(U28-Pad5) -> Net-(U25-Pad11)
- U28 pad 6: Net-(U15-Pad15) -> /Gm_pulse
- U28 pad 7: Net-(U28-Pad7) -> GND
- U28 pad 8: Net-(U15-Pad1) -> (no net)
- U28 pad 9: Net-(U28-Pad9) -> (no net)
- U29 pad 1: Net-(U29-Pad1) -> GND
- U29 pad 10: Net-(U14-Pad1) -> GND
- U29 pad 11: /Rst_clk_audm1 -> /Clk_main3
- U29 pad 13: Net-(U29-Pad13) -> /AM_db4
- U29 pad 14: Net-(U29-Pad14) -> /AM_db5
- U29 pad 16: VCC -> Net-(U29-Pad16)
- U29 pad 3: Net-(U29-Pad3) -> /AM_db0
- U29 pad 4: Net-(U29-Pad4) -> /AM_db1
- U29 pad 5: Net-(U27-Pad17) -> Net-(U29-Pad5)
- U29 pad 6: Net-(U27-Pad15) -> Net-(U29-Pad6)
- U29 pad 7: Net-(U27-Pad13) -> /AM_db2
- U29 pad 8: GND -> /AM_db3
- U29 pad 9: Net-(U27-Pad11) -> Net-(U29-Pad9)
- U3 pad 1: GND -> (no net)
- U3 pad 10: GND -> /Clk_divb11
- U3 pad 11: /Chm_2 -> Net-(U1-Pad3)
- U3 pad 12: Net-(U3-Pad12) -> /Clk_divb20
- U3 pad 13: /AM_db4 -> /Clk_divb19
- U3 pad 14: /AM_db5 -> (no net)
- U3 pad 15: Net-(U3-Pad15) -> (no net)
- U3 pad 16: Net-(U3-Pad16) -> VCC
- U3 pad 2: Net-(U3-Pad2) -> /Clk_divb17
- U3 pad 3: /AM_db0 -> /Clk_divb16
- U3 pad 4: /AM_db1 -> /Clk_divb18
- U3 pad 5: Net-(U3-Pad5) -> /Clk_divb15
- U3 pad 6: Net-(U3-Pad6) -> /Clk_divb14
- U3 pad 7: /AM_db2 -> /Clk_divb13
- U3 pad 8: /AM_db3 -> GND
- U3 pad 9: Net-(U3-Pad9) -> /Clk_divb12
- U30 pad 1: Net-(U30-Pad1) -> GND
- U30 pad 10: Net-(U15-Pad1) -> (no net)
- U30 pad 11: /Rst_clk_audm0 -> (no net)
- U30 pad 12: Net-(U30-Pad12) -> (no net)
- U30 pad 13: Net-(U30-Pad13) -> (no net)
- U30 pad 14: Net-(U30-Pad14) -> VCC
- U30 pad 2: Net-(U30-Pad2) -> GND
- U30 pad 3: Net-(U30-Pad3) -> (no net)
- U30 pad 4: Net-(U30-Pad4) -> GND
- U30 pad 5: Net-(U28-Pad17) -> GND
- U30 pad 6: Net-(U28-Pad15) -> (no net)
- U30 pad 7: Net-(U28-Pad13) -> GND
- U30 pad 8: GND -> (no net)
- U30 pad 9: Net-(U28-Pad11) -> (no net)
- U31 pad 1: Net-(U31-Pad1) -> (no net)
- U31 pad 10: /Clk_main3 -> /Clk_audv_data
- U31 pad 11: /Master_reset -> /Vrst
- U31 pad 12: Net-(U31-Pad12) -> (no net)
- U31 pad 13: Net-(U31-Pad13) -> (no net)
- U31 pad 14: Net-(U31-Pad14) -> (no net)
- U31 pad 15: Net-(U31-Pad15) -> (no net)
- U31 pad 2: Net-(U31-Pad2) -> Net-(U26-Pad30)
- U31 pad 3: Net-(U31-Pad3) -> Net-(U26-Pad2)
- U31 pad 4: Net-(U31-Pad4) -> (no net)
- U31 pad 5: /A3_aud_m -> Net-(U26-Pad3)
- U31 pad 6: /A2_aud_m -> Net-(U26-Pad29)
- U31 pad 7: /A1_aud_m -> Net-(U26-Pad28)
- U31 pad 9: /A0_aud_m -> Net-(U26-Pad4)
- U32 pad 1: GND -> (no net)
- U32 pad 10: GND -> Net-(U29-Pad15)
- U32 pad 11: /Chm_3 -> Net-(U29-Pad16)
- U32 pad 12: Net-(U23-Pad12) -> Net-(U29-Pad19)
- U32 pad 13: /AM_db12 -> VCC
- U32 pad 14: /AM_db13 -> Net-(R13-Pad2)
- U32 pad 15: Net-(U23-Pad14) -> GND
- U32 pad 16: Net-(U23-Pad16) -> Net-(C53-Pad1)
- U32 pad 2: Net-(U23-Pad3) -> Net-(R11-Pad2)
- U32 pad 3: /AM_db8 -> -12VA
- U32 pad 4: /AM_db9 -> Net-(R14-Pad2)
- U32 pad 5: Net-(U23-Pad5) -> Net-(U29-Pad2)
- U32 pad 6: Net-(U23-Pad7) -> Net-(U29-Pad5)
- U32 pad 7: /AM_db10 -> Net-(U29-Pad6)
- U32 pad 8: /AM_db11 -> Net-(U29-Pad9)
- U32 pad 9: Net-(U23-Pad9) -> Net-(U29-Pad12)
- U33 pad 1: GND -> /Maout
- U33 pad 10: GND -> Net-(C57-Pad1)
- U33 pad 11: /Chm_2 -> -12VA
- U33 pad 12: Net-(U24-Pad12) -> Net-(C59-Pad1)
- U33 pad 13: /AM_db12 -> Net-(C60-Pad1)
- U33 pad 14: /AM_db13 -> Net-(C60-Pad1)
- U33 pad 2: Net-(U24-Pad3) -> Net-(R14-Pad2)
- U33 pad 3: /AM_db8 -> GND
- U33 pad 4: /AM_db9 -> +12VA
- U33 pad 5: Net-(U24-Pad5) -> Net-(C55-Pad1)
- U33 pad 6: Net-(U24-Pad7) -> Net-(C56-Pad1)
- U33 pad 7: /AM_db10 -> Net-(C56-Pad1)
- U33 pad 8: /AM_db11 -> Net-(C58-Pad1)
- U33 pad 9: Net-(U24-Pad9) -> Net-(C58-Pad1)
- U34 pad 1: GND -> (no net)
- U34 pad 2: Net-(U27-Pad3) -> GND
- U34 pad 3: /AM_db8 -> Net-(C60-Pad1)
- U34 pad 4: /AM_db9 -> GND
- U34 pad 5: Net-(U27-Pad5) -> Net-(C61-Pad1)
- U34 pad 6: Net-(U27-Pad7) -> +12VA
- U34 pad 7: /AM_db10 -> (no net)
- U34 pad 8: /AM_db11 -> (no net)
- U4 pad 1: GND -> /Clk_divb11
- U4 pad 10: GND -> /Clk_main2
- U4 pad 11: Clk_main7 -> Net-(U1-Pad3)
- U4 pad 12: Clk_main6 -> /Clk_divb8
- U4 pad 13: Clk_main5 -> /Clk_divb7
- U4 pad 14: Clk_main4 -> /Clk_divb9
- U4 pad 15: Net-(U123-Pad10) -> /Clk_divb10
- U4 pad 16: /Clk_main2 -> VCC
- U4 pad 2: Net-(P1-Pad14) -> /Clk_divb5
- U4 pad 3: Net-(U4-Pad18) -> /Clk_divb4
- U4 pad 4: Net-(U4-Pad18) -> /Clk_divb6
- U4 pad 5: Net-(U4-Pad18) -> /Clk_divb3
- U4 pad 6: Net-(U4-Pad18) -> /Clk_divb2
- U4 pad 7: Net-(U4-Pad18) -> /Clk_divb1
- U4 pad 8: Net-(U4-Pad18) -> GND
- U4 pad 9: Net-(U4-Pad18) -> /Clk_divb0
- U5 pad 1: GND -> /Clk_gme_data
- U5 pad 10: GND -> /Clk_main2
- U5 pad 11: /Chm_1 -> GND
- U5 pad 12: Net-(U10-Pad11) -> Net-(U10-Pad27)
- U5 pad 13: /AM_db4 -> Net-(U10-Pad5)
- U5 pad 14: /AM_db5 -> Net-(U10-Pad26)
- U5 pad 15: Net-(U10-Pad13) -> Net-(U10-Pad23)
- U5 pad 16: Net-(U10-Pad15) -> VCC
- U5 pad 2: Net-(U10-Pad2) -> Net-(U10-Pad7)
- U5 pad 3: /AM_db0 -> Net-(U10-Pad8)
- U5 pad 4: /AM_db1 -> Net-(U10-Pad6)
- U5 pad 5: Net-(U10-Pad4) -> Net-(U10-Pad9)
- U5 pad 6: Net-(U10-Pad6) -> Net-(U10-Pad10)
- U5 pad 7: /AM_db2 -> /GmSelectB1
- U5 pad 8: /AM_db3 -> GND
- U5 pad 9: Net-(U10-Pad8) -> /GmSelectB0
- U6 pad 1: GND -> (no net)
- U6 pad 10: GND -> Net-(P2-Pad14)
- U6 pad 11: /Chm_0 -> /Master_reset
- U6 pad 12: Net-(U11-Pad11) -> (no net)
- U6 pad 13: /AM_db4 -> (no net)
- U6 pad 14: /AM_db5 -> (no net)
- U6 pad 15: Net-(U11-Pad13) -> (no net)
- U6 pad 16: Net-(U11-Pad15) -> VCC
- U6 pad 2: Net-(U11-Pad2) -> (no net)
- U6 pad 3: /AM_db0 -> Net-(U14-Pad2)
- U6 pad 4: /AM_db1 -> (no net)
- U6 pad 5: Net-(U11-Pad4) -> (no net)
- U6 pad 6: Net-(U11-Pad6) -> (no net)
- U6 pad 7: /AM_db2 -> (no net)
- U6 pad 8: /AM_db3 -> GND
- U6 pad 9: Net-(U11-Pad8) -> (no net)
- U7 pad 1: Net-(U18-Pad25) -> Net-(U2-Pad6)
- U7 pad 10: /A3_aud_m -> Net-(U27-Pad8)
- U7 pad 11: /M_reset -> (no net)
- U7 pad 12: Net-(U18-Pad27) -> GND
- U7 pad 13: Net-(U18-Pad5) -> GND
- U7 pad 14: Net-(U18-Pad26) -> VCC
- U7 pad 2: Net-(U18-Pad7) -> Net-(U2-Pad8)
- U7 pad 3: Net-(U18-Pad8) -> /Rst_audM
- U7 pad 4: Net-(U18-Pad6) -> /Rst_audV
- U7 pad 5: Net-(U18-Pad9) -> /GM_adress_latch
- U7 pad 6: Net-(U18-Pad10) -> Net-(U1-Pad9)
- U7 pad 7: Net-(U18-Pad11) -> GND
- U7 pad 8: GND -> /Rst_audV
- U7 pad 9: Net-(U18-Pad12) -> Net-(U27-Pad6)
- U8 pad 11: Net-(U2-Pad12) -> /GM_adress_latch
- U8 pad 12: Net-(U12-Pad3) -> Net-(U11-Pad6)
- U8 pad 13: Net-(U2-Pad15) -> /Gm_db4
- U8 pad 14: Net-(U12-Pad2) -> /Gm_db5
- U8 pad 15: Net-(U2-Pad16) -> Net-(U11-Pad7)
- U8 pad 16: Net-(U12-Pad4) -> Net-(U11-Pad8)
- U8 pad 17: Net-(U2-Pad19) -> /Gm_db6
- U8 pad 18: Net-(U12-Pad13) -> /Gm_db7
- U8 pad 19: Net-(U22-Pad2) -> Net-(U11-Pad9)
- U8 pad 2: Net-(U2-Pad2) -> Net-(U11-Pad2)
- U8 pad 3: Net-(U12-Pad9) -> /Gm_db0
- U8 pad 4: Net-(U2-Pad5) -> /Gm_db1
- U8 pad 5: Net-(U12-Pad7) -> Net-(U11-Pad3)
- U8 pad 6: Net-(U2-Pad6) -> Net-(U11-Pad4)
- U8 pad 7: Net-(U12-Pad6) -> /Gm_db2
- U8 pad 8: Net-(U2-Pad9) -> /Gm_db3
- U8 pad 9: Net-(U12-Pad5) -> Net-(U11-Pad5)
- U9 pad 1: GND -> (no net)
- U9 pad 10: GND -> Net-(U10-Pad10)
- U9 pad 11: Net-(U3-Pad12) -> /GmSelectB1
- U9 pad 12: Net-(U13-Pad3) -> /GmSelectB0
- U9 pad 13: Net-(U3-Pad15) -> /Gm_db8
- U9 pad 14: Net-(U13-Pad2) -> /Gm_db9
- U9 pad 15: Net-(U3-Pad16) -> /Gm_db10
- U9 pad 16: Net-(U13-Pad4) -> GND
- U9 pad 17: Net-(U3-Pad19) -> /Gm_db11
- U9 pad 18: Net-(U13-Pad13) -> /Gm_db12
- U9 pad 19: Net-(U22-Pad5) -> /Gm_db13
- U9 pad 2: Net-(U3-Pad2) -> Net-(U10-Pad2)
- U9 pad 20: VCC -> /Gm_db14
- U9 pad 3: Net-(U13-Pad9) -> Net-(U10-Pad3)
- U9 pad 4: Net-(U3-Pad5) -> Net-(U10-Pad4)
- U9 pad 5: Net-(U13-Pad7) -> Net-(U10-Pad5)
- U9 pad 6: Net-(U3-Pad6) -> Net-(U10-Pad6)
- U9 pad 7: Net-(U13-Pad6) -> Net-(U10-Pad7)
- U9 pad 8: Net-(U3-Pad9) -> Net-(U10-Pad8)
- U9 pad 9: Net-(U13-Pad5) -> Net-(U10-Pad9)
Routing:
- net Net-(U18-Pad23): track 71.2 -> 0.00 mm
- net Net-(U18-Pad25): track 63.7 -> 0.00 mm
- net /A3_aud_m: track 49.1 -> 0.00 mm
- net Net-(U18-Pad26): track 47.4 -> 0.00 mm
- net /A0_aud_m: track 45.0 -> 0.00 mm, vias 2 -> 0
- net Net-(U18-Pad27): track 35.1 -> 0.00 mm
- net /A1_aud_m: track 31.8 -> 0.00 mm
- net Net-(U17-Pad2): track 30.4 -> 0.00 mm
- net /A2_aud_m: track 29.8 -> 0.00 mm
- net Net-(U16-Pad2): track 29.4 -> 0.00 mm
- net Net-(U17-Pad3): track 25.1 -> 0.00 mm
- net Net-(U18-Pad7): track 24.6 -> 0.00 mm
- net Net-(U16-Pad4): track 22.0 -> 0.00 mm
- net Net-(U16-Pad3): track 22.0 -> 0.00 mm
- net Net-(U18-Pad8): track 21.5 -> 0.00 mm
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- removed copper zone on In1.Cu, net GND
- removed copper zone on In2.Cu, net VCC
Other:
- copper layers 4 -> 2

Commit message: Pcb design
Parts:
- removed C31, C34, C37, C40, C43, C46: 1µ, Capacitors_SMD:C_0805_HandSoldering
- removed C32, C33, C35, C36, C38, C39, C41, C42, C44, C45, C47, C48: 10n, Capacitors_SMD:C_0805_HandSoldering
- removed U30: 74LS21, Sockets_DIP:DIP-14__300
- C1, C14, C15, C16, C18, C19, C2, C22, C24, C25, C27, C28, C29, C30, C4, C5, C50, C69, C8, C9, P3, P4, P5, U10, U11, U12, U15, U18, U22, U23, U26, U28, U3, U32, U33, U34, U5, U6: moved to B.Cu
- C57: value 200p -> 100p
- P8: footprint Socket_Strips:Socket_Strip_Angled_1x02 -> Socket_Strips:Socket_Strip_Straight_1x02
- moved U34 283.8 mm to (21.7, 96.5), turned to 90 degrees
- moved C27 272.8 mm to (32.5, 39.3), turned to 180 degrees
- moved C28 269.1 mm to (32.5, 41.5), turned to 180 degrees
- moved C1 268.9 mm to (21.2, 16.5), turned to 90 degrees
- moved C26 268.4 mm to (26.3, 36.6), turned to 270 degrees
- moved C23 266.5 mm to (18.0, 44.4)
- moved C68 265.2 mm to (36.9, 107.2)
- moved C67 262.0 mm to (33.5, 101.2), turned to 90 degrees
- moved C65 260.7 mm to (40.9, 101.3), turned to 90 degrees
- moved C25 260.2 mm to (39.9, 41.7)
- moved C64 255.4 mm to (46.9, 94.2), turned to 90 degrees
- moved C19 253.1 mm to (40.4, 71.8), turned to 90 degrees
- moved C9 252.9 mm to (45.1, 15.2), turned to 180 degrees
- moved C63 250.4 mm to (46.9, 89.4), turned to 90 degrees
- moved R1 249.4 mm to (18.6, 40.7), turned to 180 degrees
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Connections:
- C69 pad 2: (no net) -> Net-(C69-Pad2)
- U1 pad 11: /Rst_Gam -> (no net)
- U1 pad 12: /Gwn -> GND
- U1 pad 13: /Gm_pulse -> GND
- U17 pad 1: GND -> /Gwn
- U17 pad 2: GND -> /Gm_pulse
- U17 pad 3: (no net) -> /Rst_Gam
- U19 pad 2: Net-(U19-Pad2) -> Net-(C69-Pad2)
- U22 pad 3: Net-(U19-Pad2) -> Net-(C69-Pad2)
- U28 pad 10: (no net) -> GND
- U28 pad 12: (no net) -> GND
- U28 pad 13: (no net) -> GND
- U28 pad 9: (no net) -> GND
Routing:
- net -12VA: track 0.00 -> 157.0 mm, vias 0 -> 2
- net /GM_adress_latch: track 0.00 -> 152.4 mm, vias 0 -> 5
- net /GW2: track 0.00 -> 144.7 mm, vias 0 -> 2
- net +12VA: track 0.00 -> 138.1 mm, vias 0 -> 1
- net /Clk_main3: track 0.00 -> 135.8 mm, vias 0 -> 6
- net /Master_reset: track 0.00 -> 132.5 mm, vias 0 -> 5
- net /GW1: track 0.00 -> 128.4 mm
- net Net-(U29-Pad15): track 0.00 -> 127.5 mm
- net /GW3: track 0.00 -> 122.2 mm
- net Net-(U29-Pad16): track 0.00 -> 122.0 mm
- net Net-(U29-Pad19): track 0.00 -> 119.5 mm
- net /Clk_divb14: track 0.00 -> 118.8 mm, vias 0 -> 3
- net /GW0: track 0.00 -> 114.8 mm
- net /lGm_db13: track 0.00 -> 110.3 mm
- net /lGm_db14: track 0.00 -> 109.3 mm
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- added copper zone on In1.Cu, net GND
- added copper zone on In2.Cu, net VCC
Other:
- board outline added: 100 x 100 mm
- copper layers 2 -> 4
- net class Signal added: clearance 0.16, trace_width 0.16, via_dia 0.6, via_drill 0.4
- rule trace_min: 0.2 -> 0.16

Commit message: Main pcb done
Routing:
- net GND: track 67.7 -> 1125.9 mm, vias 1 -> 24
- net VCC: track 9.58 -> 731.3 mm, vias 0 -> 18
- net /Clk_main7: track 0.00 -> 68.3 mm, vias 0 -> 6
- net /Clk_main4: track 0.00 -> 56.8 mm, vias 0 -> 3
- net /Clk_main5: track 0.00 -> 47.4 mm
- net /Clk_main6: track 0.00 -> 44.5 mm
- net /RST_GM0: track 0.00 -> 41.6 mm, vias 0 -> 1
- net /RST_GM1: track 0.00 -> 35.9 mm, vias 0 -> 2
- net /RST_GM2: track 0.00 -> 33.7 mm, vias 0 -> 1
- net /RST_GM3: track 0.00 -> 28.6 mm, vias 0 -> 2
- net Net-(U10-Pad8): track 13.2 -> 34.9 mm, vias 0 -> 3
- net Net-(U10-Pad30): track 14.3 -> 34.5 mm
- net Net-(U10-Pad6): track 13.2 -> 31.0 mm
- net /Gm_db8: track 7.77 -> 22.9 mm
- net Net-(U16-Pad2): track 0.00 -> 6.88 mm
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